File: rev2/aquarius-plus.kicad_sch (KiCad schematic)
At the start: 172 parts, among them J1 Power in, J10 FPGA spare, J11 Hand controller 2, J12 Hand controller 1, J13 ESP32 spare, J2 ESP USB Host, J3 Audio out, J4 VGA, J5 Cassette out, J6 Cassette in, J7 Expansion port, J8 Printer, J9 TF-03A, Q1 BC847C, Q2 BC847C, Q3 2N7002, SW1 SW_DPDT_x2, U1 SN74AHCT1G125DBVR, U10 ESP32-S3-WROOM-1-N4R2, U11 LDL1117S33R, U12 SN74CB3T3245PWR, U13 IS61C5128AS-25QLI, U2 SN74AHCT1G125DBVR, U3 LD1117S12, U4 SN74CB3T3245PWR, U5 MAX3221ECPWR, U6 XC6SLX9-2TQG144C, U7 Z84C0010AEG, U8 SN74CB3T3245PWR, U9 SN74CB3T3245PWR, X1 SX3M14.31818M20F30TNN

Commit message: PCB rev2-230718 Update to Use throughhole audio jacks (C2939180)
Parts:
- J3, J5, J6, J8: footprint aquarius-plus:C2884998 -> aquarius-plus:C2939180
Changed lines of the file:
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@@
       (effects (font (size 1.27 1.27)) (justify right))
     )
-    (property "Footprint" "aquarius-plus:C2884998" (at 170.18 201.93 0)
+    (property "Footprint" "aquarius-plus:C2939180" (at 170.18 201.93 0)
       (effects (font (size 1.27 1.27)) hide)
     )
@@
       (effects (font (size 1.27 1.27)) (justify right))
     )
-    (property "Footprint" "aquarius-plus:C2884998" (at 144.78 284.48 0)
+    (property "Footprint" "aquarius-plus:C2939180" (at 144.78 284.48 0)
       (effects (font (size 1.27 1.27)) hide)
     )
@@
       (effects (font (size 1.27 1.27)) (justify right))
     )
-    (property "Footprint" "aquarius-plus:C2884998" (at 113.03 313.69 0)
+    (property "Footprint" "aquarius-plus:C2939180" (at 113.03 313.69 0)
       (effects (font (size 1.27 1.27)) hide)
     )
@@
       (effects (font (size 1.27 1.27)) (justify right))
     )
-    (property "Footprint" "aquarius-plus:C2884998" (at 297.18 179.07 0)
+    (property "Footprint" "aquarius-plus:C2939180" (at 297.18 179.07 0)
       (effects (font (size 1.27 1.27)) hide)
     )
