File: mini_rev1/aquarius-plus.kicad_pcb (KiCad board)
At the start: 2 copper layers, 128 x 83 mm, 109 parts, among them J1 Power in, J10 FPGA spare, J13 ESP32 spare, J2 ESP USB Host, J3 Audio out, J4 VGA, J9 TF-03A, Q3 2N7002, SW1 SW_DPDT_x2, U10 ESP32-S3-WROOM-1-N4R2, U11 LDL1117S33R, U13 IS61C5128AL-10TLI, U3 LD1117S12, U6 XC6SLX9-2TQG144C, X1 SX3M14.31818M20F30TNN

Commit message: More Aq+ Mini vZ work...
Routing:
- net GND: track 97.5 -> 1031.4 mm, vias 156 -> 138
- net FPGA_EXP6: track 40.2 -> 41.1 mm
- net FPGA_A4: track 16.9 -> 16.4 mm
- net +5V: track 239.0 -> 238.7 mm, vias 2 -> 1
