File: mini/mini_rev1/aquarius-plus.kicad_pcb (KiCad board)
At the start: 2 copper layers, 128 x 83 mm, 109 parts, among them J1 Power in, J10 FPGA spare, J13 ESP32 spare, J2 ESP USB Host, J3 Audio out, J4 VGA, J9 TF-03A, Q3 2N7002, SW1 SW_DPDT_x2, U10 ESP32-S3-WROOM-1-N4R2, U11 LDL1117S33R, U13 IS61C5128AL-10TLI, U3 LD1117S12, U6 XC6SLX9-2TQG144C, X1 SX3M14.31818M20F30TNN

Commit message: Mini vZ rev1
Parts:
- U2: renamed from U10; footprint aquarius-plus:ESP32-S2-SOLO-N4R2 -> RF_Module:ESP32-S3-WROOM-1U
- moved U2 30.9 mm to (93.4, 68.8)
- moved R17 17.4 mm to (168.9, 52.1)
- moved #G1 17.4 mm to (178.8, 63.2)
- moved R13 17.4 mm to (161.9, 53.6)
- moved U1 17.4 mm to (129.2, 61.4)
- moved C15 17.4 mm to (127.5, 66.6)
- moved C16 17.4 mm to (133.7, 77.9)
- moved FB1 17.4 mm to (98.6, 36.9)
- moved J5 17.4 mm to (115.0, 56.6)
- moved JP4 17.4 mm to (97.3, 53.9)
- moved R1 17.4 mm to (137.7, 49.0)
- moved R27 17.4 mm to (105.4, 72.0)
- moved R30 17.4 mm to (127.5, 68.1)
- moved R32 17.4 mm to (117.6, 83.0)
- moved JP3 17.4 mm to (92.5, 44.4)
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- renumbered C7 to C1, C36 to C10, C14 to C11, C32 to C12, C30 to C14, C12 to C15, C34 to C16, C20 to C17, C38 to C18, C43 to C19, C4 to C2, C33 to C20, C42 to C21, C21 to C22, C18 to C23, C22 to C24, C37 to C25, C39 to C26, C44 to C27, C40 to C28, C19 to C29, C2 to C3, C15 to C30, C17 to C32, C16 to C33, C6 to C34, C55 to C35, C47 to C36, C48 to C37, C51 to C38, C50 to C39, C1 to C4, C52 to C40, C46 to C41, C53 to C42, C49 to C43, C35 to C44, C54 to C45, C3 to C5, C5 to C6, C58 to C7, C57 to C8, C56 to C9, D3 to D1, J3 to J2, J4 to J3, J2 to J4, J13 to J5, J9 to J6, J10 to J7, JP4 to JP2, JP2 to JP3, JP3 to JP4, Q3 to Q1, R6 to R1, R19 to R10, R9 to R12, R17 to R13, R7 to R14, R12 to R15, R8 to R16, R14 to R17, R10 to R18, R49 to R19, R5 to R2, R40 to R20, R42 to R21, R45 to R22, R68 to R23, R41 to R24, R43 to R25, R44 to R26, R38 to R27, R37 to R28, R46 to R29, R36 to R30, R47 to R31, R48 to R32, R69 to R33, R39 to R34, R16 to R5, R20 to R6, R13 to R7, R15 to R8, R21 to R9, U3 to U1, U6 to U3, U13 to U4, U11 to U5
Routing:
- net +5V: track 238.7 -> 224.1 mm
- net GND: track 1031.4 -> 1033.9 mm
- net unconnected-(U2-IO45-Pad26): track 0.00 -> 1.14 mm, vias 0 -> 1
- net ESP_USB_D-: track 76.7 -> 77.7 mm
- net ESP_USB_D+: track 78.9 -> 79.9 mm
- net unconnected-(U2-IO46/I-Pad16): track 0.00 -> 0.76 mm, vias 0 -> 1
- net ESP_EXP2: track 30.1 -> 30.7 mm
- net Net-(JP4-A): track 10.3 -> 10.8 mm
- net ESP_RTS: track 38.1 -> 38.7 mm
Other:
- board text added: "0"
- board text added: "0 mm"
- board text added: "0.01 mm"
- board text added: "0.02"
- board text added: "0.035 mm"
- board text added: "0.2000 mm / 0.0000 mm"
- board text added: "0.3000 mm"
- board text added: "1"
- board text added: "1.51 mm"
- board text added: "1.6000 mm"
- board text added: "128.0000 mm x 83.0000 mm"
- board text added: "2"
- board text added: "20240826"
- board text added: "3.3"
- board text added: "4.5"
- board text added: "B.Cu"
- board text added: "B.Mask"
- board text added: "B.Paste"
- board text added: "B.Silkscreen"
- board text added: "BOARD CHARACTERISTICS"
- board text added: "Blue"
- board text added: "Board Thickness:"
- board text added: "Board overall dimensions:"
- board text added: "Bottom Silk Screen"
- board text added: "Bottom Solder Mask"
- board text added: "Bottom Solder Paste"
- board text added: "Castellated pads:"
- board text added: "Color"
- board text added: "Copper Finish:"
- board text added: "Copper Layer Count:"
- board text added: "Dielectric 1"
- board text added: "Direct Printing"
- board text added: "Edge card connectors:"
- board text added: "Epoxy"
- board text added: "Epsilon R"
- board text added: "F.Cu"
- board text added: "F.Mask"
- board text added: "F.Paste"
- board text added: "F.Silkscreen"
- board text added: "FR4"
- board text added: "HAL lead-free"
- board text added: "Impedance Control:"
- board text added: "Layer Name"
- board text added: "Loss Tangent"
- board text added: "Material"
- board text added: "Min hole diameter:"
- board text added: "Min track/spacing:"
- board text added: "No"
- board text added: "Not specified"
- board text added: "Plated Board Edge:"
- board text added: "Thickness (mm)"
- board text added: "Top Silk Screen"
- board text added: "Top Solder Mask"
- board text added: "Top Solder Paste"
- board text added: "Type"
- board text added: "White"
- board text added: "copper"
- board text added: "core"
- board text removed: "20240822"

Commit message: Mini rev1 vZ Updates
Parts:
- renumbered C11 to C10, C30 to C11, C33 to C12, C32 to C13, C23 to C14, C29 to C15, C22 to C16, C24 to C17, C7 to C18, C8 to C19, C4 to C2, C9 to C20, C12 to C21, C14 to C22, C20 to C23, C16 to C24, C10 to C25, C18 to C26, C19 to C27, C31 to C28, C25 to C29, C26 to C30, C28 to C31, C21 to C32, C27 to C33, C43 to C38, C5 to C4, C38 to C40, C44 to C41, C40 to C42, C41 to C43, C45 to C44, C42 to C45, C2 to C5, C15 to C7, C13 to C8, C17 to C9, J4 to J2, J2 to J3, J3 to J4, J6 to J5, JP3 to JP2, JP2 to JP3, R3 to R1, R15 to R10, R5 to R11, R6 to R12, R12 to R13, R7 to R14, R13 to R15, R9 to R16, R18 to R17, R17 to R18, R30 to R19, R4 to R2, R28 to R20, R27 to R21, R19 to R22, R20 to R24, R24 to R25, R21 to R26, R25 to R27, R26 to R28, R22 to R29, R2 to R3, R29 to R30, R1 to R4, R14 to R5, R11 to R6, R8 to R7, R10 to R8, R16 to R9, U2 to U1, U1 to U2
Routing:
- net GND: track 1033.9 -> 1088.1 mm, vias 138 -> 150
Other:
- board text added: "Ext.Ant."

Commit message: Mini vZ rev1 updates
Parts:
- added C1: DNP, Capacitor_SMD:C_0603_1608Metric, F.Cu at (104.5, 48.8)
- added C2: DNP, Capacitor_SMD:C_0603_1608Metric, F.Cu at (109.0, 48.8)
- added L1: USB Choke, Inductor_SMD:L_CommonMode_Wurth_WE-CNSW-1206, F.Cu at (106.8, 48.4)
- added R1: 0, Resistor_SMD:R_0603_1608Metric, F.Cu at (106.0, 52.2)
- added R2: 0, Resistor_SMD:R_0603_1608Metric, F.Cu at (107.5, 52.2)
- added U1: IP4234CZ6, Package_TO_SOT_SMD:TSOT-23-6, F.Cu at (100.3, 47.1)
- FB1, FB2: value FerriteBead -> 220
- U2: renamed from U1; footprint RF_Module:ESP32-S3-WROOM-1U -> aquarius-plus:ESP32-S2-SOLO-N4R2
- moved U2 15.9 mm to (77.6, 69.0)
- moved C3 3.28 mm to (116.5, 49.8)
- moved JP2 2.40 mm to (92.5, 42.0), turned to 0 degrees
- moved JP1 2.40 mm to (88.2, 42.0), turned to 0 degrees
- moved FB2 2.39 mm to (122.4, 44.5)
- renumbered C8 to C10, C9 to C11, C10 to C12, C11 to C13, C12 to C14, C13 to C15, C14 to C16, C15 to C17, C16 to C18, C17 to C19, C18 to C20, C19 to C21, C20 to C22, C21 to C23, C22 to C24, C23 to C25, C24 to C26, C25 to C27, C26 to C28, C27 to C29, C1 to C3, C28 to C30, C29 to C31, C30 to C32, C31 to C33, C32 to C34, C33 to C35, C34 to C36, C35 to C37, C36 to C38, C37 to C39, C2 to C4, C38 to C40, C39 to C41, C40 to C42, C41 to C43, C42 to C44, C43 to C45, C44 to C46, C45 to C47, C3 to C5, C4 to C6, C5 to C7, C6 to C8, C7 to C9, J5 to J6, R8 to R10, R9 to R11, R10 to R12, R11 to R13, R12 to R14, R13 to R15, R14 to R16, R15 to R17, R16 to R18, R17 to R19, R18 to R20, R19 to R22, R20 to R23, R22 to R24, R23 to R25, R24 to R26, R25 to R27, R26 to R28, R27 to R29, R1 to R3, R28 to R30, R29 to R31, R30 to R32, R31 to R33, R32 to R34, R33 to R35, R34 to R36, R2 to R4, R3 to R5, R4 to R6, R5 to R7, R6 to R8, R7 to R9, U2 to U3, U3 to U4, U4 to U5, U5 to U6
Connections:
- J2 pad 2: ESP_USB_D- -> Net-(J2-D-)
- J2 pad 3: ESP_USB_D+ -> Net-(J2-D+)
- J7 pad 11: FPGA_EXP9 -> GND
- JP1 pad 2: ESP_USB_D+ -> Net-(J2-D+)
- JP2 pad 2: ESP_USB_D- -> Net-(J2-D-)
- JP3 pad 1: Net-(JP2-Pin_1) -> GND
- JP3 pad 3: GND -> Net-(JP3-Pin_3)
- JP4 pad 1: Net-(JP4-A) -> GND
- JP4 pad 2: GND -> Net-(JP4-B)
- U2 pad 27: Net-(JP4-A) -> Net-(JP4-B)
- U2 pad 37: Net-(JP2-Pin_1) -> Net-(JP3-Pin_3)
- U4 pad 50: FPGA_EXP9 -> GND
Routing:
- net ESP_USB_D+: track 79.9 -> 33.9 mm, vias 1 -> 2
- net ESP_USB_D-: track 77.7 -> 32.0 mm, vias 1 -> 2
- net FPGA_EXP9: track 34.2 -> 0.00 mm, vias 2 -> 0
- net Net-(J2-D+): track 0.00 -> 31.4 mm, vias 0 -> 2
- net Net-(J2-D-): track 0.00 -> 24.1 mm
- net GND: track 1088.1 -> 1067.0 mm, vias 150 -> 146
- net Net-(JP4-A): track 10.8 -> 0.00 mm, vias 1 -> 0
- net Net-(J1-VBUS): track 8.82 -> 19.5 mm, vias 2 -> 3
- net Net-(JP4-B): track 0.00 -> 9.78 mm, vias 0 -> 1
- net Net-(JP3-Pin_3): track 0.00 -> 7.65 mm, vias 0 -> 2
- net Net-(JP2-Pin_1): track 7.16 -> 0.00 mm, vias 1 -> 0
- net Net-(L1-Pad3): track 0.00 -> 6.76 mm
- net Net-(L1-Pad2): track 0.00 -> 5.96 mm
- net +5V: track 224.1 -> 221.3 mm
- net /USB_D+: track 10.1 -> 7.71 mm
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Other:
- board text added: "20240827"
- board text added: "Flash"
- board text added: "GND"
- board text added: "Rx"
- board text added: "Tx"
- board text removed: "20240826"
- board text removed: "Ext.Ant."

Commit message: More PCB tidying up
Parts:
- L1: footprint Inductor_SMD:L_CommonMode_Wurth_WE-CNSW-1206 -> Inductor_SMD_Wurth:WE-CNSW_08058
- turned L1 to 0 degrees
Routing:
- net Net-(L1-Pad1): track 1.76 -> 2.30 mm
- net Net-(L1-Pad4): track 1.75 -> 2.29 mm
Other:
- board text added: "20240830"
- board text removed: "20240827"
Changed lines of the file:
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@@
 	(title_block
 		(title "Aquarius+ mini vZ")
-		(date "2024-08-27")
+		(date "2024-08-30")
 		(rev "1")
 		(company "Designed by Frank van den Hoef")
@@
 		)
 	)
-	(footprint "Inductor_SMD:L_CommonMode_Wurth_WE-CNSW-1206"
+	(footprint "Inductor_SMD_Wurth:WE-CNSW_08058"
 		(layer "F.Cu")
-		(at 106.765159 48.35 90)
-		(descr "WE-CNSW SMT Common Mode Line Filter, https://www.we-online.com/components/products/datasheet/744232090.pdf")
-		(tags "common mode choke 1206 cnsw")
+		(at 106.765159 48.35)
+		(descr "WE-CNSW_08058")
+		(tags "Inductor")
 		(property "Reference" "L1"
-			(at 2.958403 0.012611 0)
-			(unlocked yes)
+			(at 0.116563 -2.484358 0)
 			(layer "F.SilkS")
 			(effects
@@
 		)
 		(property "Value" "USB Choke"
-			(at 0 3.5 90)
-			(unlocked yes)
-			(layer "F.Fab")
+			(at -1.1712 1.5288 0)
+			(layer "F.SilkS")
+			(hide yes)
 			(effects
 				(font
-					(size 1 1)
-					(thickness 0.15)
+					(size 1.27 1.27)
+					(thickness 0.254)
 				)
 			)
 		)
-		(property "Footprint" "Inductor_SMD:L_CommonMode_Wurth_WE-CNSW-1206"
-			(at 0 0 90)
-			(unlocked yes)
+		(property "Footprint" "Inductor_SMD_Wurth:WE-CNSW_08058"
+			(at 0 0 0)
 			(layer "F.Fab")
 			(hide yes)
@@
 			)
 		)
-		(property "Datasheet" "https://www.we-online.com/components/products/datasheet/744232090.pdf"
-			(at 0 0 90)
-			(unlocked yes)
+		(property "Datasheet" "https://www.we-online.com/components/products/datasheet/744231091.pdf"
+			(at 0 0 0)
 			(layer "F.Fab")
 			(hide yes)
@@
 			)
 		)
-		(property "Description" "Common mode choke, 370 mA, 125VDC, USB2.0, 111 nH"
-			(at 0 0 90)
-			(unlocked yes)
+		(property "Description" "Common mode choke, 370 mA, 125VDC, USB2.0, 131 nH"
+			(at 0 0 0)
 			(layer "F.Fab")
 			(hide yes)
@@
 		(attr smd)
 		(fp_line
-			(start -2.05 -1.05)
-			(end 1.35 -1.05)
+			(start -0.8 -1.5)
+			(end -0.8 1.5)
 			(stroke
-				(width 0.1)
-				(type default)
+				(width 0.127)
+				(type solid)
 			)
-			(layer "F.SilkS")
+			(layer "F.CrtYd")
 		)
 		(fp_line
-			(start -1.35 1.05)
-			(end 1.35 1.05)
+			(start -0.8 1.5)
+			(end 0.8 1.5)
 			(stroke
-				(width 0.1)
-				(type default)
+				(width 0.127)
+				(type solid)
 			)
-			(layer "F.SilkS")
+			(layer "F.CrtYd")
 		)
-		(fp_rect
-			(start -2.15 -1.05)
-			(end 2.15 1.05)
+		(fp_line
+			(start 0.8 -1.5)
+			(end -0.8 -1.5)
 			(stroke
-				(width 0.05)
-				(type default)
+				(width 0.127)
+				(type solid)
 			)
-			(fill none)
 			(layer "F.CrtYd")
 		)
 		(fp_line
-			(start 1.6 -0.8)
-			(end 1.6 0.8)
+			(start 0.8 1.5)
+			(end 0.8 -1.5)
 			(stroke
-				(width 0.1)
-				(type default)
+				(width 0.127)
+				(type solid)
+			)
+			(layer "F.CrtYd")
+		)
+		(fp_line
+			(start -0.6246 -1.2635)
+			(end 0.6251 -1.2635)
+			(stroke
+				(width 0.127)
+				(type solid)
 			)
 			(layer "F.Fab")
 		)
 		(fp_line
-			(start -1.1 -0.8)
-			(end 1.6 -0.8)
+			(start -0.6246 1.2874)
+			(end -0.6246 -1.2635)
 			(stroke
-				(width 0.1)
-				(type default)
+				(width 0.127)
+				(type solid)
 			)
 			(layer "F.Fab")
 		)
 		(fp_line
-			(start -1.6 -0.3)
-			(end -1.1 -0.8)
+			(start -0.4 -0.85)
+			(end -0.4 0.85)
 			(stroke
-				(width 0.1)
-				(type default)
+				(width 0.07)
+				(type solid)
 			)
 			(layer "F.Fab")
 		)
 		(fp_line
-			(start 1.6 0.8)
-			(end -1.6 0.8)
+			(start 0.4 -0.85)
+			(end 0.4 0.85)
 			(stroke
-				(width 0.1)
-				(type default)
+				(width 0.07)
+				(type solid)
 			)
 			(layer "F.Fab")
 		)
 		(fp_line
-			(start -1.6 0.8)
-			(end -1.6 -0.3)
+			(start 0.6203 1.2874)
+			(end -0.6246 1.2874)
 			(stroke
-				(width 0.1)
-				(type default)
+				(width 0.127)
+				(type solid)
+			)
+			(layer "F.Fab")
+		)
+		(fp_line
+			(start 0.6251 -1.2635)
+			(end 0.6251 1.2826)
+			(stroke
+				(width 0.127)
+				(type solid)
 			)
 			(layer "F.Fab")
 		)
 		(fp_text user "${REFERENCE}"
-			(at 0 0 90)
-			(unlocked yes)
+			(at -1.1712 1.5288 0)
 			(layer "F.Fab")
 			(effects
 				(font
-					(size 0.7 0.7)
-					(thickness 0.105)
+					(size 1.27 1.27)
+					(thickness 0.254)
 				)
 			)
 		)
-		(pad "1" smd roundrect
-			(at -1.35 -0.5 90)
-			(size 1.1 0.6)
+		(pad "1" smd rect
+			(at -0.4 0.85)
+			(size 0.4 0.9)
 			(layers "F.Cu" "F.Paste" "F.Mask")
-			(roundrect_rratio 0.2)
 			(net 161 "Net-(L1-Pad1)")
 			(pintype "passive")
-			(thermal_bridge_angle 45)
 		)
-		(pad "2" smd roundrect
-			(at 1.35 -0.5 90)
-			(size 1.1 0.6)
+		(pad "2" smd rect
+			(at -0.4 -0.85)
+			(size 0.4 0.9)
 			(layers "F.Cu" "F.Paste" "F.Mask")
-			(roundrect_rratio 0.2)
 			(net 159 "Net-(L1-Pad2)")
 			(pintype "passive")
-			(thermal_bridge_angle 45)
 		)
-		(pad "3" smd roundrect
-			(at 1.35 0.5 90)
-			(size 1.1 0.6)
+		(pad "3" smd rect
+			(at 0.4 -0.85)
+			(size 0.4 0.9)
 			(layers "F.Cu" "F.Paste" "F.Mask")
-			(roundrect_rratio 0.2)
 			(net 158 "Net-(L1-Pad3)")
 			(pintype "passive")
-			(thermal_bridge_angle 45)
 		)
-		(pad "4" smd roundrect
-			(at -1.35 0.5 90)
-			(size 1.1 0.6)
+		(pad "4" smd rect
+			(at 0.4 0.85)
+			(size 0.4 0.9)
 			(layers "F.Cu" "F.Paste" "F.Mask")
-			(roundrect_rratio 0.2)
 			(net 160 "Net-(L1-Pad4)")
 			(pintype "passive")
-			(thermal_bridge_angle 45)
 		)
-		(model "${KIPRJMOD}/step/744232090.stp"
+		(model "${KIPRJMOD}/step/744231091.stp"
 			(offset
-				(xyz 0 0 1.8)
+				(xyz -0 0 0.81)
 			)
 			(scale
@@
 			)
 			(rotate
-				(xyz -90 0 0)
+				(xyz -180 0 90)
 			)
 		)
@@
 	)
 	(gr_circle
-		(center 105.49079 50.304658)
-		(end 105.79079 50.304658)
+		(center 105.711482 50.227793)
+		(end 106.011482 50.227793)
 		(stroke
 			(width 0.15)
@@
 		)
 	)
-	(gr_text "20240827"
+	(gr_text "20240830"
 		(at 79.292947 99.120509 90)
 		(layer "F.SilkS")
@@
 	)
 	(segment
-		(start 101.261764 46)
-		(end 106.815159 46)
+		(start 107.165159 47.5)
+		(end 107.165159 46.95)
 		(width 0.3)
 		(layer "F.Cu")
@@
 	)
 	(segment
-		(start 101.249264 46.0125)
-		(end 101.261764 46)
+		(start 101.261764 46)
+		(end 101.249264 46.0125)
 		(width 0.3)
 		(layer "F.Cu")
@@
 	)
 	(segment
-		(start 106.815159 46)
-		(end 107.265159 46.45)
+		(start 106.215159 46)
+		(end 101.261764 46)
 		(width 0.3)
 		(layer "F.Cu")
@@
 	)
 	(segment
-		(start 107.265159 46.45)
-		(end 107.265159 47)
-		(width 0.2)
+		(start 107.165159 46.95)
+		(end 106.215159 46)
+		(width 0.3)
 		(layer "F.Cu")
 		(net 158)
 	)
 	(segment
-		(start 101.249264 48.2875)
-		(end 103.036764 46.5)
+		(start 105.365159 46.5)
+		(end 106.365159 47.5)
 		(width 0.3)
 		(layer "F.Cu")
@@
 	)
 	(segment
-		(start 105.765159 46.5)
-		(end 106.265159 47)
+		(start 103.036764 46.5)
+		(end 105.365159 46.5)
 		(width 0.3)
 		(layer "F.Cu")
@@
 	)
 	(segment
-		(start 103.036764 46.5)
-		(end 105.765159 46.5)
+		(start 101.249264 48.2875)
+		(end 103.036764 46.5)
 		(width 0.3)
 		(layer "F.Cu")
@@
 	)
 	(segment
-		(start 107.265159 51.115159)
-		(end 107.5 51.35)
+		(start 107.165159 49.2)
+		(end 107.165159 51.015159)
 		(width 0.3)
 		(layer "F.Cu")
@@
 	)
 	(segment
-		(start 107.265159 49.7)
-		(end 107.265159 51.115159)
+		(start 107.165159 51.015159)
+		(end 107.5 51.35)
 		(width 0.3)
 		(layer "F.Cu")
@@
 	(segment
 		(start 106 51.35)
-		(end 106.265159 51.084841)
+		(end 106.365159 50.984841)
 		(width 0.3)
 		(layer "F.Cu")
@@
 	)
 	(segment
-		(start 106.265159 51.084841)
-		(end 106.265159 49.7)
+		(start 106.365159 50.984841)
+		(end 106.365159 49.2)
 		(width 0.3)
 		(layer "F.Cu")
