File: mini/mini_rev1/aquarius-plus.kicad_pcb (KiCad board)
At the start: 2 copper layers, 128 x 83 mm, 115 parts, among them J1 Power in, J2 ESP USB Host, J3 Audio out, J4 VGA, J5 ESP32 spare, J6 TF-03A, J7 FPGA spare, Q1 2N7002, SW1 SW_DPDT_x2, U1 IP4234CZ6, U2 ESP32-S3-WROOM-1-N4R2, U3 LD1117S12, U4 XC6SLX9-2TQG144C, U5 IS61C5128AL-10TLI, U6 LDL1117S33R, X1 SX3M14.31818M20F30TNN

Commit message: Mini/vZ Updates
Routing:
- net GND: vias 146 -> 156
Other:
- board text added: "20241127"
- board text removed: "20240830"
Changed lines of the file:
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@@
 	(title_block
 		(title "Aquarius+ mini vZ")
-		(date "2024-08-30")
+		(date "2024-11-27")
 		(rev "1")
 		(company "Designed by Frank van den Hoef")
@@
 		)
 	)
-	(gr_text "20240830"
+	(gr_text "20241127"
 		(at 79.292947 99.120509 90)
 		(layer "F.SilkS")
@@
 	)
 	(via
+		(at 123.075 107)
+		(size 0.6)
+		(drill 0.3)
+		(layers "F.Cu" "B.Cu")
+		(net 2)
+	)
+	(via
 		(at 97.244483 39.910798)
 		(size 0.6)
@@
 	)
 	(via
+		(at 93.4 108.8)
+		(size 0.6)
+		(drill 0.3)
+		(layers "F.Cu" "B.Cu")
+		(net 2)
+	)
+	(via
 		(at 176.118076 76.986195)
 		(size 0.6)
@@
 	)
 	(via
+		(at 93.4 107.6)
+		(size 0.6)
+		(drill 0.3)
+		(layers "F.Cu" "B.Cu")
+		(net 2)
+	)
+	(via
 		(at 129.290024 66.595083)
 		(size 0.6)
@@
 	)
 	(via
+		(at 94.625 107.575)
+		(size 0.6)
+		(drill 0.3)
+		(layers "F.Cu" "B.Cu")
+		(net 2)
+	)
+	(via
 		(at 155.021346 65.515481)
 		(size 0.6)
@@
 	)
 	(via
+		(at 122.475 106.4)
+		(size 0.6)
+		(drill 0.3)
+		(layers "F.Cu" "B.Cu")
+		(net 2)
+	)
+	(via
 		(at 150.892947 54.020509)
 		(size 0.6)
@@
 	)
 	(via
+		(at 94.025 108.2)
+		(size 0.6)
+		(drill 0.3)
+		(layers "F.Cu" "B.Cu")
+		(net 2)
+	)
+	(via
 		(at 136.239696 47.445881)
 		(size 0.6)
@@
 	)
 	(via
+		(at 122.475 107.6)
+		(size 0.6)
+		(drill 0.3)
+		(layers "F.Cu" "B.Cu")
+		(net 2)
+	)
+	(via
 		(at 133.792947 88.220509)
 		(size 0.6)
@@
 	)
 	(via
+		(at 123.675 106.4)
+		(size 0.6)
+		(drill 0.3)
+		(layers "F.Cu" "B.Cu")
+		(net 2)
+	)
+	(via
 		(at 157.215448 79.33301)
 		(size 0.6)
@@
 	)
 	(via
+		(at 94.625 108.8)
+		(size 0.6)
+		(drill 0.3)
+		(layers "F.Cu" "B.Cu")
+		(net 2)
+	)
+	(via
 		(at 96.814743 49)
 		(size 0.6)
@@
 	)
 	(via
+		(at 123.675 107.6)
+		(size 0.6)
+		(drill 0.3)
+		(layers "F.Cu" "B.Cu")
+		(net 2)
+	)
+	(via
 		(at 163.247495 81.970512)
 		(size 0.6)
@@
 		(min_thickness 0.25)
 		(filled_areas_thickness no)
-		(fill
+		(fill yes
 			(thermal_gap 0.5)
 			(thermal_bridge_width 0.5)
