File: mini/mini_rev1/aquarius-plus.kicad_sch (KiCad schematic)
At the start: 108 parts, among them J1 Power in, J10 FPGA spare, J13 ESP32 spare, J2 ESP USB Host, J3 Audio out, J4 VGA, J9 TF-03A, Q3 2N7002, SW1 SW_DPDT_x2, U10 ESP32-S3-WROOM-1-N4R2, U11 LDL1117S33R, U13 IS61C5128AL-10TLI, U3 LD1117S12, U6 XC6SLX9-2TQG144C, X1 SX3M14.31818M20F30TNN

Commit message: Mini vZ rev1
Parts:
- U2: renamed from U10; footprint aquarius-plus:ESP32-S2-SOLO-N4R2 -> RF_Module:ESP32-S3-WROOM-1U
- renumbered C7 to C1, C36 to C10, C14 to C11, C32 to C12, C30 to C14, C12 to C15, C34 to C16, C20 to C17, C38 to C18, C43 to C19, C4 to C2, C33 to C20, C42 to C21, C21 to C22, C18 to C23, C22 to C24, C37 to C25, C39 to C26, C44 to C27, C40 to C28, C19 to C29, C2 to C3, C15 to C30, C17 to C32, C16 to C33, C6 to C34, C55 to C35, C47 to C36, C48 to C37, C51 to C38, C50 to C39, C1 to C4, C52 to C40, C46 to C41, C53 to C42, C49 to C43, C35 to C44, C54 to C45, C3 to C5, C5 to C6, C58 to C7, C57 to C8, C56 to C9, D3 to D1, J3 to J2, J4 to J3, J2 to J4, J13 to J5, J9 to J6, J10 to J7, JP4 to JP2, JP2 to JP3, JP3 to JP4, Q3 to Q1, R6 to R1, R19 to R10, R9 to R12, R17 to R13, R7 to R14, R12 to R15, R8 to R16, R14 to R17, R10 to R18, R49 to R19, R5 to R2, R40 to R20, R42 to R21, R45 to R22, R68 to R23, R41 to R24, R43 to R25, R44 to R26, R38 to R27, R37 to R28, R46 to R29, R36 to R30, R47 to R31, R48 to R32, R69 to R33, R39 to R34, R16 to R5, R20 to R6, R13 to R7, R15 to R8, R21 to R9, U3 to U1, U6 to U3, U13 to U4, U11 to U5
Other:
- note added: "Mechanical Features"
- note added: "Power Management"
- note removed: "Mounting holes"
- note removed: "Power supply"
- moved on the sheet: C1, C10, C11, C12, C13, C14, C15, C16, C17, C18, C19, C2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

Commit message: Mini rev1 vZ Updates
Parts:
- renumbered C11 to C10, C30 to C11, C33 to C12, C32 to C13, C23 to C14, C29 to C15, C22 to C16, C24 to C17, C7 to C18, C8 to C19, C4 to C2, C9 to C20, C12 to C21, C14 to C22, C20 to C23, C16 to C24, C10 to C25, C18 to C26, C19 to C27, C31 to C28, C25 to C29, C26 to C30, C28 to C31, C21 to C32, C27 to C33, C43 to C38, C5 to C4, C38 to C40, C44 to C41, C40 to C42, C41 to C43, C45 to C44, C42 to C45, C2 to C5, C15 to C7, C13 to C8, C17 to C9, J4 to J2, J2 to J3, J3 to J4, J6 to J5, JP3 to JP2, JP2 to JP3, R3 to R1, R15 to R10, R5 to R11, R6 to R12, R12 to R13, R7 to R14, R13 to R15, R9 to R16, R18 to R17, R17 to R18, R30 to R19, R4 to R2, R28 to R20, R27 to R21, R19 to R22, R20 to R24, R24 to R25, R21 to R26, R25 to R27, R26 to R28, R22 to R29, R2 to R3, R29 to R30, R1 to R4, R14 to R5, R11 to R6, R8 to R7, R10 to R8, R16 to R9, U2 to U1, U1 to U2
Connections:
- net GND: now also JP3.1 (Pin_1); no longer JP3.3 (Pin_3)
- net at U1.37 (IO43/TXD0): now also JP3.3 (Pin_3); no longer JP3.1 (Pin_1)

Commit message: Mini vZ rev1 updates
Parts:
- added C1, C2: DNP, Capacitor_SMD:C_0603_1608Metric, symbol Device:C_Small
- added L1: USB Choke, Inductor_SMD:L_CommonMode_Wurth_WE-CNSW-1206, symbol Filter:Choke_Wurth_WE-CNSW_744232090
- added R1, R2: 0, Resistor_SMD:R_0603_1608Metric, symbol Device:R
- added U1: IP4234CZ6, Package_TO_SOT_SMD:TSOT-23-6, symbol Power_Protection:IP4234CZ6
- FB1, FB2: value FerriteBead -> 220
- FID1, FID2, FID3: now not fitted
- J5, J7, JP3: now not fitted; now left out of the parts list
- U2: renamed from U1; footprint RF_Module:ESP32-S3-WROOM-1U -> aquarius-plus:ESP32-S2-SOLO-N4R2
- renumbered C8 to C10, C9 to C11, C10 to C12, C11 to C13, C12 to C14, C13 to C15, C14 to C16, C15 to C17, C16 to C18, C17 to C19, C18 to C20, C19 to C21, C20 to C22, C21 to C23, C22 to C24, C23 to C25, C24 to C26, C25 to C27, C26 to C28, C27 to C29, C1 to C3, C28 to C30, C29 to C31, C30 to C32, C31 to C33, C32 to C34, C33 to C35, C34 to C36, C35 to C37, C36 to C38, C37 to C39, C2 to C4, C38 to C40, C39 to C41, C40 to C42, C41 to C43, C42 to C44, C43 to C45, C44 to C46, C45 to C47, C3 to C5, C4 to C6, C5 to C7, C6 to C8, C7 to C9, J5 to J6, R8 to R10, R9 to R11, R10 to R12, R11 to R13, R12 to R14, R13 to R15, R14 to R16, R15 to R17, R16 to R18, R17 to R19, R18 to R20, R19 to R22, R20 to R23, R22 to R24, R23 to R25, R24 to R26, R25 to R27, R26 to R28, R27 to R29, R1 to R3, R28 to R30, R29 to R31, R30 to R32, R31 to R33, R32 to R34, R33 to R35, R34 to R36, R2 to R4, R3 to R5, R4 to R6, R5 to R7, R6 to R8, R7 to R9, U2 to U3, U3 to U4, U4 to U5, U5 to U6
Connections:
- net FPGA_EXP9 is gone; now on net GND: J7.11 (Pin_11), U4.50 (B2_IO_GCLK30)
- net ESP_USB_D+: now also C1.2, R1.2; no longer J2.3 (D+), JP1.2 (B)
- net ESP_USB_D-: now also C2.2, R2.1; no longer J2.2 (D-), JP2.2 (B)
- net GND: now also JP4.1 (A), C1.1, C2.1, U1.2 (VN); no longer JP4.2 (B)
- net at U2.27 (IO0): now also JP4.2 (B); no longer JP4.1 (A)
- net at FB1.1, J1.1 (VBUS): now also U1.5 (VP)
- new net: L1.4, R2.2
- new net: J2.2 (D-), JP2.2 (B), U1.6
- new net: L1.1, R1.1
- new net: J2.3 (D+), JP1.2 (B), U1.1
- new net: L1.2, U1.3
- new net: L1.3, U1.4
Other:
- moved on the sheet: C10, C3, C38, C39, C4, C5, C6, C7, C8, C9, FB1, FB2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

Commit message: More PCB tidying up
Parts:
- L1: footprint Inductor_SMD:L_CommonMode_Wurth_WE-CNSW-1206 -> Inductor_SMD_Wurth:WE-CNSW_08058
Changed lines of the file:
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@@
 	(title_block
 		(title "Aquarius+ mini vZ80")
-		(date "2024-08-27")
+		(date "2024-08-30")
 		(rev "1")
 		(company "Designed by Frank van den Hoef")
@@
 			)
 		)
-		(property "Footprint" "Inductor_SMD:L_CommonMode_Wurth_WE-CNSW-1206"
+		(property "Footprint" "Inductor_SMD_Wurth:WE-CNSW_08058"
 			(at 355.6 184.15 0)
 			(effects
@@
 			)
 		)
-		(property "Datasheet" "https://www.we-online.com/components/products/datasheet/744232090.pdf"
+		(property "Datasheet" "https://www.we-online.com/components/products/datasheet/744231091.pdf"
 			(at 355.6 181.61 0)
 			(effects
@@
 			)
 		)
-		(property "Description" "Common mode choke, 370 mA, 125VDC, USB2.0, 111 nH"
+		(property "Description" "Common mode choke, 370 mA, 125VDC, USB2.0, 131 nH"
 			(at 355.6 173.99 0)
 			(effects
