File: moda/rev0/aqp_moda_SD.kicad_pcb (KiCad board)
At the start: 2 copper layers, 319.5 x 146.3 mm, 207 parts, among them J1 Power in, J10 Conn_02x03_Top_Bottom, J11 Hand Controller, J12 Conn_02x10_Odd_Even, J13 ESP32 spare, J14 Conn_01x06_Socket, J15 Conn_02x10_Odd_Even, J16 Micro_SD_Card_Det1, J17 Conn_01x06_Socket, J18 Conn_01x04, J19 Conn_01x07, J2 ESP USB Host, J20 Conn_01x07, J21 Conn_02x20_Top_Bottom, J22 Conn_02x20_Top_Bottom, J23 Conn_01x03, J24 Conn_01x03, J25 KBD Matrix, J3 Audio out, J4 VGA, J5 Cassette out, J6 Cassette in, J7 Expansion port, J77 MEC5-030-01-X-RA-W1-XX-EDGE, J8 Printer, J88 MEC5-030-01-X-RA-W1-XX-SOCKET, J9 TF-03A, J99 Hand Controller, Q1 BC847C, Q2 BC847C, Q3 2N7002, SW1 SW_DPDT_x2, U1 IP4234CZ6, U10 SN74CB3T3245PWR, U11 SN74CB3T3245PWR, U12 ESP32-S3-WROOM-1-N4R2, U13 LDL1117S33R, U15 IS61C5128AL-10TLI, U2 SN74AHCT1G125DBVR, U3 PLCC-44 SMD Socket, U4 LD1117S12, U5 SN74CB3T3245PWR, U6 SN74AHCT1G125DBVR, U7 MAX3221ECPWR, U8 XC6SLX9-2TQG144C, U9 SN74CB3T3245PWR, X1 SX3M14.31818M20F30TNN

Commit message: Moda PCB updates
Parts:
- removed the C1 at (178.7, 89.6)
- removed C10, C12, C13, C14, C18, C20, C21, C22, C24, C25, C26, C27, C28, C29, C30, C31, C32, C33, C34, C37, C38, C39, C40, C41, C43, C44, C45, C46, C47, C48, C5, C51, C52, C54, C57, C58, C61, C7, C9: 100nF, Capacitor_SMD:C_0603_1608Metric
- removed C11, C15, C16, C17, C19, C23, C35, C36, C42, C49, C50, C53, C55, C56: 4.7uF, Capacitor_SMD:C_0603_1608Metric
- removed C2: DNP, Capacitor_SMD:C_0603_1608Metric
- removed C3, C8: 100uF, Capacitor_SMD:CP_Elec_6.3x7.7
- removed C4, C6: 10uF, Capacitor_SMD:C_0805_2012Metric
- removed C59: 22uF, Capacitor_SMD:C_1206_3216Metric
- removed D1, D2: 1N4148WS, Diode_SMD:D_SOD-323_HandSoldering
- removed D3: SD act., LED_THT:LED_D3.0mm_Horizontal_O1.27mm_Z2.0mm
- removed FB1, FB2: 220, Inductor_SMD:L_0603_1608Metric
- removed the H1 at (72.0, 73.8)
- removed the H1 at (293.5, 93.5)
- removed the H1 at (121.0, 73.8)
- removed the H1 at (144.4, 153.3)
- removed the H1 at (362.5, 153.0)
- removed the H1 at (362.5, 93.5)
- removed the H1 at (241.9, 153.3)
- removed the H1 at (294.0, 153.0)
- removed the H1 at (275.4, 73.8)
- removed the H1 at (144.4, 73.8)
- removed the H2 at (278.4, 209.7)
- removed the H2 at (278.5, 188.7)
- removed H3 (x2), H4 (x2): MountingHole, MountingHole:MountingHole_3.2mm_M3
- removed the J1 at (156.2, 70.8)
- removed J10: Conn_02x03_Top_Bottom, Connector_PinSocket_2.54mm:PinSocket_2x03_P2.54mm_Vertical
- removed J11, J99: Hand Controller, Connector_Dsub:DSUB-9_Male_Horizontal_P2.77x2.84mm_EdgePinOffset9.90mm_Housed_MountingHolesOffset11.32mm
- removed J12, J15: Conn_02x10_Odd_Even, Connector_IDC:IDC-Header_2x10_P2.54mm_Vertical
- removed J13: ESP32 spare, Connector_PinHeader_2.54mm:PinHeader_2x07_P2.54mm_Vertical
- removed J14, J17: Conn_01x06_Socket, Connector_PinHeader_2.54mm:PinHeader_1x06_P2.54mm_Vertical
- removed J18: Conn_01x04, Connector_PinHeader_2.54mm:PinHeader_1x04_P2.54mm_Vertical
- removed J19: Conn_01x07, Connector_PinHeader_2.54mm:PinHeader_1x07_P2.54mm_Vertical
- removed the J2 at (179.7, 80.2)
- removed J21: Conn_02x20_Top_Bottom, Connector_IDC:IDC-Header_2x20_P2.54mm_Vertical
- removed the J22 at (304.7, 208.7)
- removed J23, J24: Conn_01x03, Connector_PinSocket_2.54mm:PinSocket_1x03_P2.54mm_Vertical
- removed J25: KBD Matrix, Connector_PinHeader_2.54mm:PinHeader_2x04_P2.54mm_Vertical
- removed J3: Audio out, aquarius-plus:C2939180
- removed J4: VGA, aquarius-plus:ICD15S13E4GV00LF
- removed J5: Cassette out, aquarius-plus:C2939180
- removed J6: Cassette in, aquarius-plus:C2939180
- removed J7: Expansion port, aquarius-plus:CR22A-44D-2.54DSA(70)
- removed J77: MEC5-030-01-X-RA-W1-XX-EDGE, samtec-mec5-30:SAMTEC_MEC5-030-01-X-RA-W1-XX-EDGE
- removed J8: Printer, aquarius-plus:C2939180
- removed J88: MEC5-030-01-X-RA-W1-XX-SOCKET, samtec-mec5-30:SAMTEC_MEC5-030-01-X-RA-W1-XX
- removed JP1, JP2: Pin Header, Connector_PinHeader_2.54mm:PinHeader_1x02_P2.54mm_Vertical
- removed JP3: vZ80 Enabled, Jumper:SolderJumper-2_P1.3mm_Bridged_RoundedPad1.0x1.5mm
- removed JP4: DBG, Connector_PinHeader_2.54mm:PinHeader_1x03_P2.54mm_Vertical
- removed JP5: Bootloader, Connector_PinHeader_2.54mm:PinHeader_1x02_P2.54mm_Vertical
- removed L1: USB Choke, Inductor_SMD_Wurth:WE-CNSW_08058
- removed the Q1 at (94.8, 87.3)
- removed Q2: BC847C, Package_TO_SOT_SMD:SOT-23
- removed the R1 at (115.7, 87.0)
- removed the R10 at (217.3, 89.8)
- removed R11, R15, R18: 536, Resistor_SMD:R_0603_1608Metric
- removed R12, R13, R20: 2150, Resistor_SMD:R_0603_1608Metric
- removed R14, R17: 1070, Resistor_SMD:R_0603_1608Metric
- removed R16, R19: 4300, Resistor_SMD:R_0603_1608Metric
- removed the R2 at (114.2, 87.0)
- removed R21, R22: 820, Resistor_SMD:R_0603_1608Metric
- removed R23, R24, R25, R26, R27, R28: 1k, Resistor_SMD:R_0603_1608Metric
- removed R29: 82, Resistor_SMD:R_0603_1608Metric
- removed the R3 at (182.1, 86.9)
- removed R30, R31: 47k, Resistor_SMD:R_0603_1608Metric
- removed R32, R39, R70: 220, Resistor_SMD:R_0603_1608Metric
- removed R33: 220k, Resistor_SMD:R_0603_1608Metric
- removed R34, R35: 4.7k, Resistor_SMD:R_0603_1608Metric
- removed R36: 2.2k, Resistor_SMD:R_0603_1608Metric
- removed R37, R52, R53, R54, R55, R56, R57, R58, R59, R60, R61, R62, R63, R64, R65, R66, R67, R68, R69: 100, Resistor_SMD:R_0603_1608Metric
- removed R38, R40: 0, Resistor_SMD:R_0603_1608Metric
- removed the R4 at (182.1, 88.4)
- removed R41: 10k, Resistor_SMD:R_0603_1608Metric
- removed the R5 at (193.6, 85.1)
- removed the R6 at (200.9, 85.1)
- removed the R7 at (196.6, 85.1)
- removed the R8 at (203.9, 85.1)
- removed the R9 at (217.3, 92.6)
- removed SW1: SW_DPDT_x2, Button_Switch_THT:SW_E-Switch_EG2219_DPDT_Angled
- removed U1: IP4234CZ6, Package_TO_SOT_SMD:SC-74-6_1.55x2.9mm_P0.95mm
- removed U10, U11, U5, U9: SN74CB3T3245PWR, Package_SO:TSSOP-20_4.4x6.5mm_P0.65mm
- removed U12: ESP32-S3-WROOM-1-N4R2, aquarius-plus:ESP32-S2-SOLO-N4R2
- removed U13: LDL1117S33R, Package_TO_SOT_SMD:SOT-223-3_TabPin2
- removed U15: IS61C5128AL-10TLI, Package_SO:TSOP-II-44_10.16x18.41mm_P0.8mm
- removed U2, U6: SN74AHCT1G125DBVR, Package_TO_SOT_SMD:SOT-23-5
- removed U3: PLCC-44 SMD Socket, Package_LCC:PLCC-44_SMD-Socket
- removed U4: LD1117S12, Package_TO_SOT_SMD:SOT-223-3_TabPin2
- removed U7: MAX3221ECPWR, Package_SO:TSSOP-16_4.4x5mm_P0.65mm
- removed U8: XC6SLX9-2TQG144C, Package_QFP:TQFP-144_20x20mm_P0.5mm
- removed X1: SX3M14.31818M20F30TNN, Oscillator:Oscillator_SMD_SeikoEpson_SG8002CE-4Pin_3.2x2.5mm
- moved H2 142.4 mm to (227.9, 137.5), turned to 90 degrees
- moved J22 116.0 mm to (206.7, 133.2), turned to 0 degrees
- moved R9 108.5 mm to (215.8, 112.7), turned to 90 degrees
- moved R10 106.7 mm to (214.3, 112.7), turned to -90 degrees
- moved R8 105.0 mm to (212.9, 112.7), turned to -90 degrees
- moved H1 102.7 mm to (185.9, 137.5), turned to 90 degrees
- moved R7 102.3 mm to (210.7, 112.7), turned to -90 degrees
- moved J2 100.4 mm to (206.7, 116.3), turned to 0 degrees
- moved J1 100.4 mm to (220.5, 102.9), turned to -90 degrees
- moved R6 100.3 mm to (209.0, 112.7), turned to -90 degrees
- moved C1 96.3 mm to (205.7, 112.7), turned to 90 degrees
- moved R5 93.3 mm to (203.1, 112.7), turned to -90 degrees
- moved R4 89.6 mm to (199.9, 112.7), turned to -90 degrees
- moved R3 87.7 mm to (198.2, 112.7), turned to -90 degrees
- moved R2 85.9 mm to (196.6, 112.7), turned to 90 degrees
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- renumbered C60 to C1, H1 to H2, J20 to J1, J9 to J2, J16 to J22, Q3 to Q1, R42 to R1, R50 to R10, R43 to R2, R44 to R3, R45 to R4, R46 to R5, R47 to R6, R48 to R7, R49 to R8, R51 to R9
Routing:
- net GND: track 899.9 -> 0.00 mm, vias 186 -> 0
- net +3V3: track 504.7 -> 0.00 mm, vias 17 -> 0
- net +5V: track 410.1 -> 0.00 mm, vias 22 -> 0
- net FPGA_RD#: track 175.8 -> 0.00 mm, vias 8 -> 0
- net CASSETTE_OUT: track 165.6 -> 0.00 mm, vias 7 -> 0
- net FPGA_INT#: track 120.4 -> 0.00 mm, vias 7 -> 0
- net FPGA_MREQ#: track 119.3 -> 0.00 mm, vias 7 -> 0
- net FPGA_BUSREQ#: track 116.4 -> 0.00 mm, vias 7 -> 0
- net FPGA_IORQ#: track 115.8 -> 0.00 mm, vias 2 -> 0
- net +1V2: track 113.8 -> 0.00 mm, vias 7 -> 0
- net FPGA_WR#: track 112.7 -> 0.00 mm, vias 2 -> 0
- net FPGA_RESET#: track 109.0 -> 0.00 mm, vias 2 -> 0
- net FPGA_BUSACK#: track 105.4 -> 0.00 mm, vias 2 -> 0
- net VBUS: track 101.4 -> 0.00 mm, vias 1 -> 0
- net BUSREQ#: track 100.9 -> 0.00 mm, vias 8 -> 0
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Other:
- board size 319.5 x 146.3 mm -> 51.9 x 44.4 mm
- board text added: "CD"
- board text added: "MISO"
- board text added: "MOSI"
- board text added: "Moda - SD Card Board"
- board text added: "Next Generation Z80-Based"
- board text added: "Retro Computer System"
- board text added: "SCK"
- board text added: "SSEL"
- board text added: "WP"
- board text removed: "+"
- board text removed: "-"
- board text removed: "1.2V"
- board text removed: "20240918"
- board text removed: "3.3V"
- board text removed: "512KB RAM"
- board text removed: "Audio Out"
- board text removed: "BLU"
- board text removed: "Cartridge Port"
- board text removed: "Cassette & Printer"
- board text removed: "Cassette On"
- board text removed: "Cassette Out"
- board text removed: "D+"
- board text removed: "D-"
- board text removed: "Debug"
- board text removed: "Designed in 2022/2023 by Frank van den Hoef"
- board text removed: "ESP32 Spares"
- board text removed: "ESP32 Wi-Fi and Storage"
- board text removed: "Expansion Bus Card"
- board text removed: "FPGA"
- board text removed: "FPGA Spares"
- board text removed: "Flash"
- board text removed: "GRN"
- board text removed: "HS"
- board text removed: "Hand Controller 1"
- board text removed: "Hand Controller 2"
- board text removed: "Hand Controllers"
- board text removed: "KBD Matrix"
- board text removed: "Moda"
- board text removed: "Next Generation Z80-Based Retro Computer System"
- board text removed: "OFF"
- board text removed: "ON"
- board text removed: "Power"
- board text removed: "Printer"
- board text removed: "RED"
- board text removed: "Rx"
- board text removed: "Tx"
- board text removed: "USB KBD"
- board text removed: "VGA"
- board text removed: "VS"
- board text removed: "Z80 CPU"
- board text removed: "Z80 Card"
- board text removed: "vZ"
