File: moda/rev0/aqp_moda_Z80.kicad_pcb (KiCad board)
At the start: 2 copper layers, 319.5 x 146.3 mm, 207 parts, among them J1 Power in, J10 Conn_02x03_Top_Bottom, J11 Hand Controller, J12 Conn_02x10_Odd_Even, J13 ESP32 spare, J14 Conn_01x06_Socket, J15 Conn_02x10_Odd_Even, J16 Micro_SD_Card_Det1, J17 Conn_01x06_Socket, J18 Conn_01x04, J19 Conn_01x07, J2 ESP USB Host, J20 Conn_01x07, J21 Conn_02x20_Top_Bottom, J22 Conn_02x20_Top_Bottom, J23 Conn_01x03, J24 Conn_01x03, J25 KBD Matrix, J3 Audio out, J4 VGA, J5 Cassette out, J6 Cassette in, J7 Expansion port, J77 MEC5-030-01-X-RA-W1-XX-EDGE, J8 Printer, J88 MEC5-030-01-X-RA-W1-XX-SOCKET, J9 TF-03A, J99 Hand Controller, Q1 BC847C, Q2 BC847C, Q3 2N7002, SW1 SW_DPDT_x2, U1 IP4234CZ6, U10 SN74CB3T3245PWR, U11 SN74CB3T3245PWR, U12 ESP32-S3-WROOM-1-N4R2, U13 LDL1117S33R, U15 IS61C5128AL-10TLI, U2 SN74AHCT1G125DBVR, U3 PLCC-44 SMD Socket, U4 LD1117S12, U5 SN74CB3T3245PWR, U6 SN74AHCT1G125DBVR, U7 MAX3221ECPWR, U8 XC6SLX9-2TQG144C, U9 SN74CB3T3245PWR, X1 SX3M14.31818M20F30TNN

Commit message: Moda PCB updates
Parts:
- removed the C1 at (178.7, 89.6)
- removed C11, C15, C16, C17, C19, C23, C35, C36, C42, C49, C50, C53, C55, C56, C60: 4.7uF, Capacitor_SMD:C_0603_1608Metric
- removed C14, C18, C20, C21, C22, C24, C25, C26, C27, C28, C29, C32, C33, C34, C37, C38, C39, C40, C41, C43, C44, C47, C48, C51, C52, C54, C57, C58, C61, C9: 100nF, Capacitor_SMD:C_0603_1608Metric
- removed the C2 at (178.7, 85.6)
- removed the C3 at (191.1, 92.7)
- removed the C4 at (191.9, 85.1)
- removed the C5 at (195.1, 85.1)
- removed C59: 22uF, Capacitor_SMD:C_1206_3216Metric
- removed the C6 at (199.1, 85.1)
- removed the C7 at (202.4, 85.1)
- removed C8: 100uF, Capacitor_SMD:CP_Elec_6.3x7.7
- removed D1, D2: 1N4148WS, Diode_SMD:D_SOD-323_HandSoldering
- removed D3: SD act., LED_THT:LED_D3.0mm_Horizontal_O1.27mm_Z2.0mm
- removed FB1, FB2: 220, Inductor_SMD:L_0603_1608Metric
- removed the H1 at (72.0, 73.8)
- removed the H1 at (86.5, 111.9)
- removed the H1 at (121.0, 73.8)
- removed the H1 at (144.4, 153.3)
- removed the H1 at (86.5, 153.9)
- removed the H1 at (241.9, 153.3)
- removed the H1 at (275.4, 73.8)
- removed the H1 at (144.4, 73.8)
- removed the H2 at (278.4, 209.7)
- removed the H2 at (278.5, 188.7)
- removed the H3 at (154.0, 198.0)
- removed the H3 at (229.5, 198.0)
- removed the H4 at (379.4, 209.7)
- removed the H4 at (379.5, 188.7)
- removed the J1 at (156.2, 70.8)
- removed J10: Conn_02x03_Top_Bottom, Connector_PinSocket_2.54mm:PinSocket_2x03_P2.54mm_Vertical
- removed J11, J99: Hand Controller, Connector_Dsub:DSUB-9_Male_Horizontal_P2.77x2.84mm_EdgePinOffset9.90mm_Housed_MountingHolesOffset11.32mm
- removed J12, J15: Conn_02x10_Odd_Even, Connector_IDC:IDC-Header_2x10_P2.54mm_Vertical
- removed J13: ESP32 spare, Connector_PinHeader_2.54mm:PinHeader_2x07_P2.54mm_Vertical
- removed J14, J17: Conn_01x06_Socket, Connector_PinHeader_2.54mm:PinHeader_1x06_P2.54mm_Vertical
- removed J16: Micro_SD_Card_Det1, Connector_Card:microSD_HC_Hirose_DM3AT-SF-PEJM5
- removed J18: Conn_01x04, Connector_PinHeader_2.54mm:PinHeader_1x04_P2.54mm_Vertical
- removed J19, J20: Conn_01x07, Connector_PinHeader_2.54mm:PinHeader_1x07_P2.54mm_Vertical
- removed the J2 at (179.7, 80.2)
- removed J22: Conn_02x20_Top_Bottom, Connector_IDC:IDC-Header_2x20_P2.54mm_Vertical
- removed J24: Conn_01x03, Connector_PinSocket_2.54mm:PinSocket_1x03_P2.54mm_Vertical
- removed J25: KBD Matrix, Connector_PinHeader_2.54mm:PinHeader_2x04_P2.54mm_Vertical
- removed the J3 at (197.7, 74.3)
- removed J4: VGA, aquarius-plus:ICD15S13E4GV00LF
- removed J5: Cassette out, aquarius-plus:C2939180
- removed J6: Cassette in, aquarius-plus:C2939180
- removed J7: Expansion port, aquarius-plus:CR22A-44D-2.54DSA(70)
- removed J77: MEC5-030-01-X-RA-W1-XX-EDGE, samtec-mec5-30:SAMTEC_MEC5-030-01-X-RA-W1-XX-EDGE
- removed J8: Printer, aquarius-plus:C2939180
- removed J9: TF-03A, aquarius-plus:TF-03A
- removed JP1, JP2: Pin Header, Connector_PinHeader_2.54mm:PinHeader_1x02_P2.54mm_Vertical
- removed JP3: vZ80 Enabled, Jumper:SolderJumper-2_P1.3mm_Bridged_RoundedPad1.0x1.5mm
- removed JP4: DBG, Connector_PinHeader_2.54mm:PinHeader_1x03_P2.54mm_Vertical
- removed JP5: Bootloader, Connector_PinHeader_2.54mm:PinHeader_1x02_P2.54mm_Vertical
- removed L1: USB Choke, Inductor_SMD_Wurth:WE-CNSW_08058
- removed Q1, Q2: BC847C, Package_TO_SOT_SMD:SOT-23
- removed Q3: 2N7002, Package_TO_SOT_SMD:SOT-23
- removed the R1 at (115.7, 87.0)
- removed R10, R14, R17: 1070, Resistor_SMD:R_0603_1608Metric
- removed R11, R15, R18: 536, Resistor_SMD:R_0603_1608Metric
- removed R12, R13, R20: 2150, Resistor_SMD:R_0603_1608Metric
- removed R16, R19, R9: 4300, Resistor_SMD:R_0603_1608Metric
- removed the R2 at (114.2, 87.0)
- removed R21, R22: 820, Resistor_SMD:R_0603_1608Metric
- removed R29: 82, Resistor_SMD:R_0603_1608Metric
- removed the R3 at (182.1, 86.9)
- removed R30, R31: 47k, Resistor_SMD:R_0603_1608Metric
- removed R32, R39, R70: 220, Resistor_SMD:R_0603_1608Metric
- removed R33: 220k, Resistor_SMD:R_0603_1608Metric
- removed R34, R35: 4.7k, Resistor_SMD:R_0603_1608Metric
- removed R36: 2.2k, Resistor_SMD:R_0603_1608Metric
- removed R37, R44, R46, R48, R49, R52, R53, R54, R55, R56, R57, R58, R59, R60, R61, R62, R63, R64, R65, R66, R67, R68, R69: 100, Resistor_SMD:R_0603_1608Metric
- removed R38, R40: 0, Resistor_SMD:R_0603_1608Metric
- removed the R4 at (182.1, 88.4)
- removed R41, R42, R43, R45, R47, R50, R51: 10k, Resistor_SMD:R_0603_1608Metric
- removed the R5 at (193.6, 85.1)
- removed the R6 at (200.9, 85.1)
- removed R7, R8: 330, Resistor_SMD:R_0603_1608Metric
- removed SW1: SW_DPDT_x2, Button_Switch_THT:SW_E-Switch_EG2219_DPDT_Angled
- removed the U1 at (171.1, 87.8)
- removed U12: ESP32-S3-WROOM-1-N4R2, aquarius-plus:ESP32-S2-SOLO-N4R2
- removed U13: LDL1117S33R, Package_TO_SOT_SMD:SOT-223-3_TabPin2
- removed U15: IS61C5128AL-10TLI, Package_SO:TSOP-II-44_10.16x18.41mm_P0.8mm
- removed the U4 at (180.0, 129.7)
- removed the U7 at (81.4, 88.4)
- removed U8: XC6SLX9-2TQG144C, Package_QFP:TQFP-144_20x20mm_P0.5mm
- removed X1: SX3M14.31818M20F30TNN, Oscillator:Oscillator_SMD_SeikoEpson_SG8002CE-4Pin_3.2x2.5mm
- J3: renamed from J21; value Conn_02x20_Top_Bottom -> IDC_02x20
- moved C5 127.5 mm to (207.1, 130.4)
- moved C7 127.5 mm to (201.2, 137.7)
- moved J3 127.5 mm to (176.6, 155.2)
- moved R3 127.5 mm to (220.0, 109.9)
- moved R4 127.5 mm to (220.0, 112.9)
- moved U4 127.5 mm to (228.7, 118.1)
- moved C1 127.5 mm to (186.8, 103.2)
- moved C2 127.5 mm to (186.8, 115.2)
- moved C3 127.5 mm to (226.4, 122.4)
- moved C4 127.5 mm to (186.8, 127.2)
- moved C6 127.5 mm to (175.2, 137.6)
- moved H1 127.5 mm to (166.0, 95.2)
- moved H2 127.5 mm to (235.0, 95.2)
- moved H3 127.5 mm to (166.5, 154.7)
- moved H4 127.5 mm to (235.0, 154.7)
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- renumbered C30 to C1, C45 to C2, C13 to C3, C46 to C4, C31 to C5, C10 to C6, C12 to C7, H1 to H2, H1 to H3, H1 to H4, J88 to J1, J23 to J2, R24 to R1, R23 to R2, R25 to R3, R27 to R4, R28 to R5, R26 to R6, U9 to U1, U10 to U2, U5 to U4, U11 to U5, U2 to U6, U6 to U7
Routing:
- net GND: track 899.9 -> 23.7 mm, vias 186 -> 76
- net +5V: track 410.1 -> 16.8 mm, vias 22 -> 13
- net +3V3: track 504.7 -> 153.0 mm, vias 17 -> 7
- net CASSETTE_OUT: track 165.6 -> 39.1 mm, vias 7 -> 2
- net +1V2: track 113.8 -> 0.00 mm, vias 7 -> 0
- net VBUS: track 101.4 -> 0.00 mm, vias 1 -> 0
- net FPGA_RD#: track 175.8 -> 86.4 mm, vias 8 -> 4
- net CASSETTE_IN: track 80.7 -> 0.00 mm, vias 3 -> 0
- net PRINTER_IN: track 77.1 -> 0.00 mm, vias 3 -> 0
- net PRINTER_OUT: track 77.0 -> 0.00 mm, vias 3 -> 0
- net FPGA_A9: track 89.8 -> 14.1 mm, vias 3 -> 0
- net FPGA_A6: track 94.9 -> 19.7 mm, vias 6 -> 2
- net FPGA_A8: track 92.6 -> 17.6 mm, vias 6 -> 2
- net FPGA_A10: track 94.2 -> 19.2 mm, vias 8 -> 2
- net FPGA_A5: track 89.2 -> 14.4 mm, vias 3 -> 0
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- added copper zone on In2.Cu, net +5V
- added copper zone on In1.Cu, net GND
Other:
- board size 319.5 x 146.3 mm -> 84.3 x 69.8 mm
- copper layers 2 -> 4
- board text added: "+5V"
- board text added: "Computer System"
- board text added: "Expansion Bus Card Connector"
- board text added: "Moda - Z80 CPU Card"
- board text added: "Next Generation Z80-Based"
- board text added: "Requires a Z80 CMOS CPU PLCC44 10MHZ or higher Z84C0010VEC"
- board text removed: "+"
- board text removed: "-"
- board text removed: "1.2V"
- board text removed: "20240918"
- board text removed: "3.3V"
- board text removed: "512KB RAM"
- board text removed: "Audio Out"
- board text removed: "BLU"
- board text removed: "Cartridge Port"
- board text removed: "Cassette & Printer"
- board text removed: "Cassette On"
- board text removed: "Cassette Out"
- board text removed: "D+"
- board text removed: "D-"
- board text removed: "Debug"
- board text removed: "Designed in 2022/2023 by Frank van den Hoef"
- board text removed: "ESP32 Spares"
- board text removed: "ESP32 Wi-Fi and Storage"
- board text removed: "Expansion Bus Card"
- board text removed: "FPGA"
- board text removed: "FPGA Spares"
- board text removed: "Flash"
- board text removed: "GRN"
- board text removed: "HS"
- board text removed: "Hand Controller 1"
- board text removed: "Hand Controller 2"
- board text removed: "Hand Controllers"
- board text removed: "KBD Matrix"
- board text removed: "Moda"
- board text removed: "Next Generation Z80-Based Retro Computer System"
- board text removed: "OFF"
- board text removed: "ON"
- board text removed: "Power"
- board text removed: "Printer"
- board text removed: "RED"
- board text removed: "Rx"
- board text removed: "SD Card"
- board text removed: "Tx"
- board text removed: "USB KBD"
- board text removed: "VGA"
- board text removed: "VS"
- board text removed: "Z80 Card"
- board text removed: "vZ"
