File: moda/rev0/aqp_moda_Z80.kicad_sch (KiCad schematic)
At the start: 193 parts, among them J1 Power in, J10 Conn_02x03_Top_Bottom, J11 Hand Controller, J12 Conn_02x10_Odd_Even, J13 ESP32 spare, J14 Conn_01x06_Socket, J15 Conn_02x10_Odd_Even, J16 Micro_SD_Card_Det1, J17 Conn_01x06_Socket, J18 Conn_01x04, J19 Conn_01x07, J2 ESP USB Host, J20 Conn_01x07, J21 Conn_02x20_Top_Bottom, J22 Conn_02x20_Top_Bottom, J23 Conn_01x03, J24 Conn_01x03, J25 KBD Matrix, J3 Audio out, J4 VGA, J5 Cassette out, J6 Cassette in, J7 Expansion port, J77 MEC5-030-01-X-RA-W1-XX-EDGE, J8 Printer, J88 MEC5-030-01-X-RA-W1-XX-SOCKET, J9 TF-03A, J99 Hand Controller, Q1 BC847C, Q2 BC847C, Q3 2N7002, SW1 SW_DPDT_x2, U1 IP4234CZ6, U10 SN74CB3T3245PWR, U11 SN74CB3T3245PWR, U12 ESP32-S3-WROOM-1-N4R2, U13 LDL1117S33R, U15 IS61C5128AL-10TLI, U2 SN74AHCT1G125DBVR, U3 PLCC-44 SMD Socket, U4 LD1117S12, U5 SN74CB3T3245PWR, U6 SN74AHCT1G125DBVR, U7 MAX3221ECPWR, U8 XC6SLX9-2TQG144C, U9 SN74CB3T3245PWR, X1 SX3M14.31818M20F30TNN

Commit message: Moda PCB updates
Parts:
- removed C1, C2: DNP, Capacitor_SMD:C_0603_1608Metric, symbol Device:C_Small
- removed C11, C15, C16, C17, C19, C23, C35, C36, C42, C49, C50, C53, C55, C56, C60: 4.7uF, Capacitor_SMD:C_0603_1608Metric, symbol Device:C_Small
- removed C14, C18, C20, C21, C22, C24, C25, C26, C27, C28, C29, C32, C33, C34, C37, C38, C39, C40, C41, C43, C44, C47, C48, C5, C51, C52, C54, C57, C58, C61, C7, C9: 100nF, Capacitor_SMD:C_0603_1608Metric, symbol Device:C_Small
- removed C3, C8: 100uF, Capacitor_SMD:CP_Elec_6.3x7.7, symbol Device:C_Polarized_Small
- removed C4, C6: 10uF, Capacitor_SMD:C_0805_2012Metric, symbol Device:C_Small
- removed C59: 22uF, Capacitor_SMD:C_1206_3216Metric, symbol Device:C_Small
- removed D1, D2: 1N4148WS, Diode_SMD:D_SOD-323_HandSoldering, symbol Diode:1N4148WS
- removed D3: SD act., LED_THT:LED_D3.0mm_Horizontal_O1.27mm_Z2.0mm, symbol Device:LED
- removed FB1, FB2: 220, Inductor_SMD:L_0603_1608Metric, symbol Device:FerriteBead
- removed J1: Power in, aquarius-plus:AMPHENOL_10118194-0001LF, symbol Connector:USB_B_Micro
- removed J10: Conn_02x03_Top_Bottom, Connector_PinSocket_2.54mm:PinSocket_2x03_P2.54mm_Vertical, symbol Connector_Generic:Conn_02x03_Top_Bottom
- removed J11, J99: Hand Controller, Connector_Dsub:DSUB-9_Male_Horizontal_P2.77x2.84mm_EdgePinOffset9.90mm_Housed_MountingHolesOffset11.32mm, symbol Connector:DB9_Male_MountingHoles
- removed J12, J15: Conn_02x10_Odd_Even, Connector_IDC:IDC-Header_2x10_P2.54mm_Vertical, symbol Connector_Generic:Conn_02x10_Odd_Even
- removed J13: ESP32 spare, Connector_PinHeader_2.54mm:PinHeader_2x07_P2.54mm_Vertical, symbol Connector_Generic:Conn_02x07_Odd_Even
- removed J14, J17: Conn_01x06_Socket, Connector_PinHeader_2.54mm:PinHeader_1x06_P2.54mm_Vertical, symbol Connector:Conn_01x06_Socket
- removed J16: Micro_SD_Card_Det1, Connector_Card:microSD_HC_Hirose_DM3AT-SF-PEJM5, symbol Connector:Micro_SD_Card_Det1
- removed J18: Conn_01x04, Connector_PinHeader_2.54mm:PinHeader_1x04_P2.54mm_Vertical, symbol Connector_Generic:Conn_01x04
- removed J19, J20: Conn_01x07, Connector_PinHeader_2.54mm:PinHeader_1x07_P2.54mm_Vertical, symbol Connector_Generic:Conn_01x07
- removed J2: ESP USB Host, Connector_USB:USB_A_Molex_67643_Horizontal, symbol Connector:USB_A
- removed J21: Conn_02x20_Top_Bottom, Connector_IDC:IDC-Header_2x20_P2.54mm_Vertical, symbol Connector_Generic:Conn_02x20_Top_Bottom
- removed J24: Conn_01x03, Connector_PinSocket_2.54mm:PinSocket_1x03_P2.54mm_Vertical, symbol Connector_Generic:Conn_01x03
- removed J25: KBD Matrix, Connector_PinHeader_2.54mm:PinHeader_2x04_P2.54mm_Vertical, symbol Connector_Generic:Conn_02x04_Top_Bottom
- removed J3: Audio out, aquarius-plus:C2939180, symbol Connector:AudioJack3
- removed J4: VGA, aquarius-plus:ICD15S13E4GV00LF, symbol Connector:DB15_Female_HighDensity_MountingHoles
- removed J5: Cassette out, aquarius-plus:C2939180, symbol Connector:AudioJack3
- removed J6: Cassette in, aquarius-plus:C2939180, symbol Connector:AudioJack3
- removed J7: Expansion port, aquarius-plus:CR22A-44D-2.54DSA(70), symbol Connector_Generic:Conn_02x22_Odd_Even
- removed J77: MEC5-030-01-X-RA-W1-XX-EDGE, samtec-mec5-30:SAMTEC_MEC5-030-01-X-RA-W1-XX-EDGE, symbol samtec-mec5-30:MEC5-030-01-X-RA-W1-XX
- removed J8: Printer, aquarius-plus:C2939180, symbol Connector:AudioJack3
- removed J9: TF-03A, aquarius-plus:TF-03A, symbol Connector:SD_Card
- removed JP1, JP2: Pin Header, Connector_PinHeader_2.54mm:PinHeader_1x02_P2.54mm_Vertical, symbol Jumper:Jumper_2_Open
- removed JP3: vZ80 Enabled, Jumper:SolderJumper-2_P1.3mm_Bridged_RoundedPad1.0x1.5mm, symbol Jumper:SolderJumper_2_Bridged
- removed JP4: DBG, Connector_PinHeader_2.54mm:PinHeader_1x03_P2.54mm_Vertical, symbol Connector_Generic:Conn_01x03
- removed JP5: Bootloader, Connector_PinHeader_2.54mm:PinHeader_1x02_P2.54mm_Vertical, symbol Jumper:Jumper_2_Open
- removed L1: USB Choke, Inductor_SMD_Wurth:WE-CNSW_08058, symbol Filter:Choke_Wurth_WE-CNSW_744232090
- removed Q1, Q2: BC847C, Package_TO_SOT_SMD:SOT-23, symbol Transistor_BJT:BC847
- removed Q3: 2N7002, Package_TO_SOT_SMD:SOT-23, symbol Transistor_FET:2N7002
- removed R1, R41, R42, R43, R45, R47, R50, R51: 10k, Resistor_SMD:R_0603_1608Metric, symbol Device:R
- removed R10, R14, R17: 1070, Resistor_SMD:R_0603_1608Metric, symbol Device:R
- removed R11, R15, R18: 536, Resistor_SMD:R_0603_1608Metric, symbol Device:R
- removed R12, R13, R20: 2150, Resistor_SMD:R_0603_1608Metric, symbol Device:R
- removed R16, R19, R9: 4300, Resistor_SMD:R_0603_1608Metric, symbol Device:R
- removed R2, R37, R44, R46, R48, R49, R52, R53, R54, R55, R56, R57, R58, R59, R60, R61, R62, R63, R64, R65, R66, R67, R68, R69: 100, Resistor_SMD:R_0603_1608Metric, symbol Device:R
- removed R21, R22: 820, Resistor_SMD:R_0603_1608Metric, symbol Device:R
- removed R29: 82, Resistor_SMD:R_0603_1608Metric, symbol Device:R
- removed R3, R38, R4, R40: 0, Resistor_SMD:R_0603_1608Metric, symbol Device:R
- removed R30, R31: 47k, Resistor_SMD:R_0603_1608Metric, symbol Device:R
- removed R32, R39, R70: 220, Resistor_SMD:R_0603_1608Metric, symbol Device:R
- removed R33: 220k, Resistor_SMD:R_0603_1608Metric, symbol Device:R
- removed R34, R35: 4.7k, Resistor_SMD:R_0603_1608Metric, symbol Device:R
- removed R36: 2.2k, Resistor_SMD:R_0603_1608Metric, symbol Device:R
- removed R5, R6: 150, Resistor_SMD:R_0603_1608Metric, symbol Device:R
- removed R7, R8: 330, Resistor_SMD:R_0603_1608Metric, symbol Device:R
- removed SW1: SW_DPDT_x2, Button_Switch_THT:SW_E-Switch_EG2219_DPDT_Angled, symbol Switch:SW_DPDT_x2
- removed U1: IP4234CZ6, Package_TO_SOT_SMD:SC-74-6_1.55x2.9mm_P0.95mm, symbol Power_Protection:IP4234CZ6
- removed U12: ESP32-S3-WROOM-1-N4R2, aquarius-plus:ESP32-S2-SOLO-N4R2, symbol aquarius-plus:ESP32-S3-WROOM-1-N4R2
- removed U13: LDL1117S33R, Package_TO_SOT_SMD:SOT-223-3_TabPin2, symbol Regulator_Linear:AP1117-33
- removed U15: IS61C5128AL-10TLI, Package_SO:TSOP-II-44_10.16x18.41mm_P0.8mm, symbol Memory_RAM:IS61C5128AL-10TLI
- removed U4: LD1117S12, Package_TO_SOT_SMD:SOT-223-3_TabPin2, symbol Regulator_Linear:AP1117-33
- removed U7: MAX3221ECPWR, Package_SO:TSSOP-16_4.4x5mm_P0.65mm, symbol Interface_UART:MAX3221
- removed U8: XC6SLX9-2TQG144C, Package_QFP:TQFP-144_20x20mm_P0.5mm, symbol aquarius-plus:XC6SLX9-2TQG144C
- removed X1: SX3M14.31818M20F30TNN, Oscillator:Oscillator_SMD_SeikoEpson_SG8002CE-4Pin_3.2x2.5mm, symbol Oscillator:SG-5032CAN
- J3: renamed from J22; value Conn_02x20_Top_Bottom -> IDC_02x20
- renumbered C30 to C1, C45 to C2, C13 to C3, C46 to C4, C31 to C5, C10 to C6, C12 to C7, J88 to J1, J23 to J2, R24 to R1, R23 to R2, R25 to R3, R27 to R4, R28 to R5, R26 to R6, U9 to U1, U10 to U2, U5 to U4, U11 to U5, U2 to U6, U6 to U7
Connections:
- no-connect marks 25 -> 0
Other:
- note added: "Expansion Port Connector"
- note added: "Level Translation"
- note added: "Mounting Holes"
- note added: "Samtec Connector"
- note added: "Various Pullups"
- note added: "Z80 Processor"
- note removed: "512KB SRAM"
- note removed: "Activity LED"
- note removed: "Audio output"
- note removed: "Cartridge port"
- note removed: "Cassette interface"
- note removed: "ESP32"
- note removed: "FPGA"
- note removed: "Handcontroller interface"
- note removed: "Mainboard Connector"
- note removed: "Mounting holes"
- note removed: "Power supply"
- note removed: "Secure Digital card interface"
- note removed: "Serial printer port"
- note removed: "Spare ESP32 pins"
- note removed: "Spare FPGA pins"
- note removed: "Subboard Connector"
- note removed: "System clock (14.31818MHz)"
- note removed: "USB host / slave via ESP32"
- note removed: "VGA interface"
- note removed: "Various pullups"
- note removed: "Z80 processor"
- title: Aquarius+ Standard -> Aquarius+ Moda: Z80 Daughterboard
- moved on the sheet: C1, C2, C3, C4, C5, C6, C7, H1, H2, H3, H4, J1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
