File: moda/rev0/aqp_moda_Main.kicad_pcb (KiCad board)
At the start: 2 copper layers, 319.5 x 146.3 mm, 207 parts, among them J1 Power in, J10 Conn_02x03_Top_Bottom, J11 Hand Controller, J12 Conn_02x10_Odd_Even, J13 ESP32 spare, J14 Conn_01x06_Socket, J15 Conn_02x10_Odd_Even, J16 Micro_SD_Card_Det1, J17 Conn_01x06_Socket, J18 Conn_01x04, J19 Conn_01x07, J2 ESP USB Host, J20 Conn_01x07, J21 Conn_02x20_Top_Bottom, J22 Conn_02x20_Top_Bottom, J23 Conn_01x03, J24 Conn_01x03, J25 KBD Matrix, J3 Audio out, J4 VGA, J5 Cassette out, J6 Cassette in, J7 Expansion port, J77 MEC5-030-01-X-RA-W1-XX-EDGE, J8 Printer, J88 MEC5-030-01-X-RA-W1-XX-SOCKET, J9 TF-03A, J99 Hand Controller, Q1 BC847C, Q2 BC847C, Q3 2N7002, SW1 SW_DPDT_x2, U1 IP4234CZ6, U10 SN74CB3T3245PWR, U11 SN74CB3T3245PWR, U12 ESP32-S3-WROOM-1-N4R2, U13 LDL1117S33R, U15 IS61C5128AL-10TLI, U2 SN74AHCT1G125DBVR, U3 PLCC-44 SMD Socket, U4 LD1117S12, U5 SN74CB3T3245PWR, U6 SN74AHCT1G125DBVR, U7 MAX3221ECPWR, U8 XC6SLX9-2TQG144C, U9 SN74CB3T3245PWR, X1 SX3M14.31818M20F30TNN

Commit message: Moda PCB updates
Parts:
- removed the C10 at (302.7, 135.9)
- removed the C11 at (89.8, 87.1)
- removed the C12 at (328.7, 136.0)
- removed the C13 at (353.9, 120.7)
- removed the C14 at (75.4, 86.2)
- removed the C15 at (86.0, 87.1)
- removed the C27 at (75.4, 87.7)
- removed the C28 at (75.4, 90.6)
- removed the C29 at (75.4, 89.1)
- removed the C30 at (314.3, 101.5)
- removed the C31 at (334.6, 128.7)
- removed the C45 at (314.3, 113.5)
- removed the C46 at (314.3, 125.5)
- removed C60: 4.7uF, Capacitor_SMD:C_0603_1608Metric
- removed the C9 at (111.2, 87.0)
- removed the D1 at (101.2, 87.1)
- removed D2: 1N4148WS, Diode_SMD:D_SOD-323_HandSoldering
- removed the H1 at (72.0, 73.8)
- removed the H1 at (86.5, 111.9)
- removed the H1 at (293.5, 93.5)
- removed the H1 at (121.0, 73.8)
- removed the H1 at (362.5, 153.0)
- removed the H1 at (362.5, 93.5)
- removed the H1 at (86.5, 153.9)
- removed the H1 at (294.0, 153.0)
- removed the H2 at (278.4, 209.7)
- removed the H2 at (278.5, 188.7)
- removed the H3 at (154.0, 198.0)
- removed the H3 at (229.5, 198.0)
- removed the H4 at (379.4, 209.7)
- removed the H4 at (379.5, 188.7)
- removed the J11 at (169.2, 189.9)
- removed J15: Conn_02x10_Odd_Even, Connector_IDC:IDC-Header_2x10_P2.54mm_Vertical
- removed J16: Micro_SD_Card_Det1, Connector_Card:microSD_HC_Hirose_DM3AT-SF-PEJM5
- removed J17: Conn_01x06_Socket, Connector_PinHeader_2.54mm:PinHeader_1x06_P2.54mm_Vertical
- removed J20: Conn_01x07, Connector_PinHeader_2.54mm:PinHeader_1x07_P2.54mm_Vertical
- removed J21: Conn_02x20_Top_Bottom, Connector_IDC:IDC-Header_2x20_P2.54mm_Vertical
- removed the J22 at (304.7, 208.7)
- removed J23, J24: Conn_01x03, Connector_PinSocket_2.54mm:PinSocket_1x03_P2.54mm_Vertical
- removed the J6 at (96.5, 74.2)
- removed the J7 at (328.9, 191.3)
- removed the J8 at (81.5, 74.2)
- removed J88: MEC5-030-01-X-RA-W1-XX-SOCKET, samtec-mec5-30:SAMTEC_MEC5-030-01-X-RA-W1-XX
- removed the J9 at (107.7, 132.8)
- removed J99: Hand Controller, Connector_Dsub:DSUB-9_Male_Horizontal_P2.77x2.84mm_EdgePinOffset9.90mm_Housed_MountingHolesOffset11.32mm
- removed Q1, Q2: BC847C, Package_TO_SOT_SMD:SOT-23
- removed Q3: 2N7002, Package_TO_SOT_SMD:SOT-23
- removed the R1 at (115.7, 87.0)
- removed the R2 at (114.2, 87.0)
- removed the R23 at (341.4, 102.2)
- removed the R24 at (338.4, 102.2)
- removed the R25 at (347.5, 108.2)
- removed the R26 at (347.5, 122.7)
- removed R27, R28: 1k, Resistor_SMD:R_0603_1608Metric
- removed R29: 82, Resistor_SMD:R_0603_1608Metric
- removed R30, R31: 47k, Resistor_SMD:R_0603_1608Metric
- removed R32: 220, Resistor_SMD:R_0603_1608Metric
- removed R33: 220k, Resistor_SMD:R_0603_1608Metric
- removed R34, R35: 4.7k, Resistor_SMD:R_0603_1608Metric
- removed R36: 2.2k, Resistor_SMD:R_0603_1608Metric
- removed R42, R43, R45, R47, R50, R51: 10k, Resistor_SMD:R_0603_1608Metric
- removed R44, R46, R48, R49, R52, R53, R54, R55, R56, R57, R58, R59, R60, R61, R62, R63, R64, R65, R66, R67, R68, R69: 100, Resistor_SMD:R_0603_1608Metric
- removed U10, U11, U9: SN74CB3T3245PWR, Package_SO:TSSOP-20_4.4x6.5mm_P0.65mm
- removed the U2 at (302.2, 138.4)
- removed the U3 at (334.2, 115.5)
- removed the U5 at (356.2, 116.4)
- removed the U6 at (328.1, 138.4)
- removed U7: MAX3221ECPWR, Package_SO:TSSOP-16_4.4x5mm_P0.65mm
- added J10: Conn_01x02_Pin, Connector_PinHeader_2.54mm:PinHeader_1x02_P2.54mm_Vertical, F.Cu at (142.7, 145.1)
- D1: renamed from D3; value SD act. -> LED; footprint LED_THT:LED_D3.0mm_Horizontal_O1.27mm_Z2.0mm -> LED_SMD:LED_0805_2012Metric
- J5: value Cassette out -> Conn_01x02; footprint aquarius-plus:C2939180 -> Connector_PinHeader_2.54mm:PinHeader_1x02_P2.54mm_Horizontal
- moved J5 157.3 mm to (268.5, 81.9)
- moved D1 8.03 mm to (146.7, 135.0), turned to 180 degrees
- moved J11 2.64 mm to (167.0, 139.7)
- moved J8 1.76 mm to (201.7, 94.0)
- moved J22 0.68 mm to (180.0, 73.7)
- moved R26 0.22 mm to (146.6, 145.1)
- renumbered C2 to C1, C56 to C10, C32 to C11, C39 to C12, C40 to C13, C33 to C14, C35 to C15, C36 to C16, C34 to C17, C19 to C18, C18 to C19, C1 to C2, C21 to C20, C22 to C21, C20 to C22, C25 to C23, C23 to C25, C59 to C27, C58 to C28, C16 to C29, C4 to C3, C17 to C30, C47 to C31, C50 to C32, C48 to C33, C49 to C34, C51 to C35, C52 to C36, C54 to C37, C53 to C38, C42 to C39, C5 to C4, C44 to C40, C43 to C41, C41 to C42, C37 to C43, C38 to C44, C61 to C45, C57 to C46, C6 to C5, C7 to C6, C3 to C7, C55 to C9, H1 to H2, H1 to H3, H1 to H4, J13 to J11, J19 to J12, J12 to J13, J18 to J22, J14 to J6, J10 to J7, J25 to J8, J77 to J9, JP4 to JP3, JP5 to JP4, JP3 to JP5, R3 to R1, R9 to R10, R15 to R11, R14 to R12, R16 to R14, R18 to R15, R17 to R16, R20 to R17, R19 to R18, R21 to R19, R4 to R2, R22 to R20, R40 to R21, R39 to R22, R41 to R23, R37 to R24, R38 to R25, R70 to R26, R5 to R3, R7 to R4, R6 to R5, R8 to R6, R11 to R7, R10 to R8, R12 to R9, U12 to U2, U13 to U3, U8 to U5, U15 to U6
Connections:
- J12 pad 1: unconnected-(J19-Pin_1-Pad1) -> GND
- J12 pad 2: unconnected-(J19-Pin_2-Pad2) -> SD_SSEL#
- J12 pad 3: unconnected-(J19-Pin_3-Pad3) -> SD_MOSI
- J12 pad 4: unconnected-(J19-Pin_4-Pad4) -> SD_SCK
- J12 pad 5: unconnected-(J19-Pin_5-Pad5) -> SD_MISO
- J12 pad 6: unconnected-(J19-Pin_6-Pad6) -> SD_CD
- J12 pad 7: unconnected-(J19-Pin_7-Pad7) -> SD_WP#
Routing:
- net GND: track 899.9 -> 148.2 mm, vias 186 -> 105
- net +3V3: track 504.7 -> 231.0 mm, vias 17 -> 25
- net +5V: track 410.1 -> 167.8 mm, vias 22 -> 5
- net BUSREQ#: track 100.9 -> 0.00 mm, vias 8 -> 0
- net RESET#: track 100.9 -> 0.00 mm, vias 5 -> 0
- net FPGA_INT#: track 120.4 -> 32.6 mm, vias 7 -> 3
- net INT#: track 86.6 -> 0.00 mm, vias 5 -> 0
- net FPGA_RD#: track 175.8 -> 89.5 mm, vias 8 -> 4
- net FPGA_BUSREQ#: track 116.4 -> 30.9 mm, vias 7 -> 3
- net FPGA_MREQ#: track 119.3 -> 34.4 mm, vias 7 -> 3
- net FPGA_IORQ#: track 115.8 -> 33.3 mm
- net FPGA_WR#: track 112.7 -> 32.4 mm
- net FPGA_RESET#: track 109.0 -> 30.8 mm
- net M1#: track 76.1 -> 0.00 mm, vias 1 -> 0
- net FPGA_BUSACK#: track 105.4 -> 29.4 mm
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- added copper zone on F.Cu, net +1V2
- added copper zone on In2.Cu, net +3V3
- added copper zone on In1.Cu, net GND
Other:
- board size 319.5 x 146.3 mm -> 141 x 89.5 mm
- copper layers 2 -> 4
- board text added: "+3V3"
- board text added: "Based on Aquarius+ by Frank van den Hoef"
- board text added: "CD"
- board text added: "CIn"
- board text added: "COut"
- board text added: "Cut to Disable vZ80"
- board text added: "Designed in 2024 by Sean Harrington"
- board text added: "Do not use both!"
- board text added: "HC1"
- board text added: "HC2"
- board text added: "MISO"
- board text added: "MOSI"
- board text added: "Moda - Mainboard"
- board text added: "Next Generation Z80-Based"
- board text added: "PIn"
- board text added: "POut"
- board text added: "Remote LED"
- board text added: "Remote Power Switch"
- board text added: "Retro Computer System"
- board text added: "SCK"
- board text added: "SSEL"
- board text added: "Stereo Audio Out"
- board text added: "WP"
- board text removed: "Audio Out"
- board text removed: "Cartridge Port"
- board text removed: "Cassette On"
- board text removed: "Cassette Out"
- board text removed: "Designed in 2022/2023 by Frank van den Hoef"
- board text removed: "Expansion Bus Card"
- board text removed: "Hand Controller 1"
- board text removed: "Hand Controller 2"
- board text removed: "Moda"
- board text removed: "Next Generation Z80-Based Retro Computer System"
- board text removed: "Printer"
- board text removed: "Z80 CPU"
- board text removed: "vZ"

Commit message: Moda PCB tweaks.
Connections:
- J10 pad 1: Net-(D1-A) -> GND
- J10 pad 2: GND -> Net-(D1-A)
- J11 pad 1: +3V3 -> GND
- J11 pad 13: GND -> +3V3
- J13 pad 10: unconnected-(J13-Pin_10-Pad10) -> GND
- J13 pad 11: unconnected-(J13-Pin_11-Pad11) -> GND
- J6 pad 1: CASSETTE_OUT -> GND
- J6 pad 6: GND -> CASSETTE_OUT
- J7 pad 1: +3V3 -> GND
- J7 pad 3: GND -> +3V3
- J8 pad 1: +5V -> GND
- J8 pad 2: GND -> +5V
- J8 pad 5: +3V3 -> KBD-FirstCol
- J8 pad 6: KBD-FirstCol -> +3V3
Routing:
- net +3V3: track 231.0 -> 270.8 mm, vias 25 -> 27
- net GND: track 148.2 -> 160.4 mm, vias 105 -> 121
- net CASSETTE_OUT: track 126.5 -> 116.6 mm
- net +5V: track 167.8 -> 173.8 mm
- net Net-(D1-A): track 13.3 -> 14.3 mm
