File: moda/rev0/aqp_moda_Main.kicad_sch (KiCad schematic)
At the start: 193 parts, among them J1 Power in, J10 Conn_02x03_Top_Bottom, J11 Hand Controller, J12 Conn_02x10_Odd_Even, J13 ESP32 spare, J14 Conn_01x06_Socket, J15 Conn_02x10_Odd_Even, J16 Micro_SD_Card_Det1, J17 Conn_01x06_Socket, J18 Conn_01x04, J19 Conn_01x07, J2 ESP USB Host, J20 Conn_01x07, J21 Conn_02x20_Top_Bottom, J22 Conn_02x20_Top_Bottom, J23 Conn_01x03, J24 Conn_01x03, J25 KBD Matrix, J3 Audio out, J4 VGA, J5 Cassette out, J6 Cassette in, J7 Expansion port, J77 MEC5-030-01-X-RA-W1-XX-EDGE, J8 Printer, J88 MEC5-030-01-X-RA-W1-XX-SOCKET, J9 TF-03A, J99 Hand Controller, Q1 BC847C, Q2 BC847C, Q3 2N7002, SW1 SW_DPDT_x2, U1 IP4234CZ6, U10 SN74CB3T3245PWR, U11 SN74CB3T3245PWR, U12 ESP32-S3-WROOM-1-N4R2, U13 LDL1117S33R, U15 IS61C5128AL-10TLI, U2 SN74AHCT1G125DBVR, U3 PLCC-44 SMD Socket, U4 LD1117S12, U5 SN74CB3T3245PWR, U6 SN74AHCT1G125DBVR, U7 MAX3221ECPWR, U8 XC6SLX9-2TQG144C, U9 SN74CB3T3245PWR, X1 SX3M14.31818M20F30TNN

Commit message: Moda PCB updates
Parts:
- removed C10, C12, C13, C14, C27, C28, C29, C30, C31, C45, C46, C9: 100nF, Capacitor_SMD:C_0603_1608Metric, symbol Device:C_Small
- removed C11, C15, C60: 4.7uF, Capacitor_SMD:C_0603_1608Metric, symbol Device:C_Small
- removed D1, D2: 1N4148WS, Diode_SMD:D_SOD-323_HandSoldering, symbol Diode:1N4148WS
- removed D3: SD act., LED_THT:LED_D3.0mm_Horizontal_O1.27mm_Z2.0mm, symbol Device:LED
- removed J11, J99: Hand Controller, Connector_Dsub:DSUB-9_Male_Horizontal_P2.77x2.84mm_EdgePinOffset9.90mm_Housed_MountingHolesOffset11.32mm, symbol Connector:DB9_Male_MountingHoles
- removed J15: Conn_02x10_Odd_Even, Connector_IDC:IDC-Header_2x10_P2.54mm_Vertical, symbol Connector_Generic:Conn_02x10_Odd_Even
- removed J16: Micro_SD_Card_Det1, Connector_Card:microSD_HC_Hirose_DM3AT-SF-PEJM5, symbol Connector:Micro_SD_Card_Det1
- removed J17: Conn_01x06_Socket, Connector_PinHeader_2.54mm:PinHeader_1x06_P2.54mm_Vertical, symbol Connector:Conn_01x06_Socket
- removed J20: Conn_01x07, Connector_PinHeader_2.54mm:PinHeader_1x07_P2.54mm_Vertical, symbol Connector_Generic:Conn_01x07
- removed J21, J22: Conn_02x20_Top_Bottom, Connector_IDC:IDC-Header_2x20_P2.54mm_Vertical, symbol Connector_Generic:Conn_02x20_Top_Bottom
- removed J23, J24: Conn_01x03, Connector_PinSocket_2.54mm:PinSocket_1x03_P2.54mm_Vertical, symbol Connector_Generic:Conn_01x03
- removed J5: Cassette out, aquarius-plus:C2939180, symbol Connector:AudioJack3
- removed J6: Cassette in, aquarius-plus:C2939180, symbol Connector:AudioJack3
- removed J7: Expansion port, aquarius-plus:CR22A-44D-2.54DSA(70), symbol Connector_Generic:Conn_02x22_Odd_Even
- removed J8: Printer, aquarius-plus:C2939180, symbol Connector:AudioJack3
- removed J88: MEC5-030-01-X-RA-W1-XX-SOCKET, samtec-mec5-30:SAMTEC_MEC5-030-01-X-RA-W1-XX, symbol samtec-mec5-30:MEC5-030-01-X-RA-W1-XX
- removed J9: TF-03A, aquarius-plus:TF-03A, symbol Connector:SD_Card
- removed JP3: vZ80 Enabled, Jumper:SolderJumper-2_P1.3mm_Bridged_RoundedPad1.0x1.5mm, symbol Jumper:SolderJumper_2_Bridged
- removed Q1, Q2: BC847C, Package_TO_SOT_SMD:SOT-23, symbol Transistor_BJT:BC847
- removed Q3: 2N7002, Package_TO_SOT_SMD:SOT-23, symbol Transistor_FET:2N7002
- removed R1, R42, R43, R45, R47, R50, R51: 10k, Resistor_SMD:R_0603_1608Metric, symbol Device:R
- removed R2, R44, R46, R48, R49, R52, R53, R54, R55, R56, R57, R58, R59, R60, R61, R62, R63, R64, R65, R66, R67, R68, R69: 100, Resistor_SMD:R_0603_1608Metric, symbol Device:R
- removed R23, R24, R25, R26, R27, R28: 1k, Resistor_SMD:R_0603_1608Metric, symbol Device:R
- removed R29: 82, Resistor_SMD:R_0603_1608Metric, symbol Device:R
- removed R30, R31: 47k, Resistor_SMD:R_0603_1608Metric, symbol Device:R
- removed R32: 220, Resistor_SMD:R_0603_1608Metric, symbol Device:R
- removed R33: 220k, Resistor_SMD:R_0603_1608Metric, symbol Device:R
- removed R34, R35: 4.7k, Resistor_SMD:R_0603_1608Metric, symbol Device:R
- removed R36: 2.2k, Resistor_SMD:R_0603_1608Metric, symbol Device:R
- removed U10, U11, U5, U9: SN74CB3T3245PWR, Package_SO:TSSOP-20_4.4x6.5mm_P0.65mm, symbol aquarius-plus:SN74CB3T3245PWR
- removed U2, U6: SN74AHCT1G125DBVR, Package_TO_SOT_SMD:SOT-23-5, symbol 74xGxx:74AHCT1G125
- removed U3: PLCC-44 SMD Socket, Package_LCC:PLCC-44_SMD-Socket, symbol aquarius-plus:Z84C3008VEG
- removed U7: MAX3221ECPWR, Package_SO:TSSOP-16_4.4x5mm_P0.65mm, symbol Interface_UART:MAX3221
- added D1: LED, LED_SMD:LED_0805_2012Metric, symbol Device:LED
- added J10: Conn_01x02_Pin, Connector_PinHeader_2.54mm:PinHeader_1x02_P2.54mm_Vertical, symbol Connector:Conn_01x02_Pin
- added J5: Conn_01x02, Connector_PinHeader_2.54mm:PinHeader_1x02_P2.54mm_Horizontal, symbol Connector_Generic:Conn_01x02
- added JP5: vZ80 Enabled, Jumper:SolderJumper-2_P1.3mm_Bridged_RoundedPad1.0x1.5mm, symbol Jumper:SolderJumper_2_Bridged
- J13: renamed from J12; now not fitted; now left out of the parts list
- J22: renamed from J18; now not fitted; now left out of the parts list
- J6: renamed from J14; now not fitted; now left out of the parts list
- J8: renamed from J25; now not fitted; now left out of the parts list
- renumbered C2 to C1, C56 to C10, C32 to C11, C39 to C12, C40 to C13, C33 to C14, C35 to C15, C36 to C16, C34 to C17, C19 to C18, C18 to C19, C1 to C2, C21 to C20, C22 to C21, C20 to C22, C25 to C23, C23 to C25, C59 to C27, C58 to C28, C16 to C29, C4 to C3, C17 to C30, C47 to C31, C50 to C32, C48 to C33, C49 to C34, C51 to C35, C52 to C36, C54 to C37, C53 to C38, C42 to C39, C5 to C4, C44 to C40, C43 to C41, C41 to C42, C37 to C43, C38 to C44, C61 to C45, C57 to C46, C6 to C5, C7 to C6, C3 to C7, C55 to C9, J13 to J11, J19 to J12, J10 to J7, J77 to J9, JP4 to JP3, JP5 to JP4, R3 to R1, R9 to R10, R15 to R11, R14 to R12, R16 to R14, R18 to R15, R17 to R16, R20 to R17, R19 to R18, R21 to R19, R4 to R2, R22 to R20, R40 to R21, R39 to R22, R41 to R23, R37 to R24, R38 to R25, R70 to R26, R5 to R3, R7 to R4, R6 to R5, R8 to R6, R11 to R7, R10 to R8, R12 to R9, U12 to U2, U13 to U3, U8 to U5, U15 to U6
Connections:
- net +5V: now also J5.2 (Pin_2)
- net GND: now also J12.1 (Pin_1), D1.1 (K), J10.2 (Pin_2), JP5.1 (A)
- net SD_CD: now also J12.6 (Pin_6)
- net SD_MISO: now also J12.5 (Pin_5)
- net SD_MOSI: now also J12.3 (Pin_3)
- net SD_SCK: now also J12.4 (Pin_4)
- net SD_SSEL#: now also J12.2 (Pin_2)
- net SD_WP#: now also J12.7 (Pin_7)
- net VBUS: now also J5.1 (Pin_1)
- net vZ80 Sense: now also JP5.2 (B)
- net at R26.2: now also D1.2 (A), J10.1 (Pin_1)
- no-connect marks 25 -> 39
Other:
- note removed: "Cartridge port"
- note removed: "Cassette interface"
- note removed: "Handcontroller interface"
- note removed: "Level translation"
- note removed: "Secure Digital card interface"
- note removed: "Serial printer port"
- note removed: "Subboard Connector"
- note removed: "Various pullups"
- note removed: "Z80 processor"
- moved on the sheet: C29, C9, J12, R26

Commit message: Moda PCB tweaks.
Connections:
- net +3V3: now also J11.13 (Pin_13), J7.3 (Pin_3), J8.6 (Pin_6); no longer J11.1 (Pin_1), J7.1 (Pin_1), J8.5 (Pin_5)
- net +5V: now also J8.2 (Pin_2); no longer J8.1 (Pin_1)
- net CASSETTE_OUT: now also J6.6 (Pin_6); no longer J6.1 (Pin_1)
- net GND: now also J10.1 (Pin_1), J11.1 (Pin_1), J13.10 (Pin_10), J13.11 (Pin_11), J6.1 (Pin_1), J7.1 (Pin_1), J8.1 (Pin_1); no longer J10.2 (Pin_2), J11.13 (Pin_13), J6.6 (Pin_6), J7.3 (Pin_3), J8.2 (Pin_2)
- net KBD-FirstCol: now also J8.5 (Pin_5); no longer J8.6 (Pin_6)
- net at D1.2 (A), R26.2: now also J10.2 (Pin_2); no longer J10.1 (Pin_1)
- no-connect marks 39 -> 37
