File: standard/rev3/aquarius-plus.kicad_pcb (KiCad board)
At the start: 2 copper layers, 167 x 115 mm, 174 parts, among them J1 Power in, J10 FPGA spare, J11 Hand controller 2, J12 Hand controller 1, J13 ESP32 spare, J2 ESP USB Host, J3 Audio out, J4 VGA, J5 Cassette out, J6 Cassette in, J7 Expansion port, J8 Printer, J9 TF-03A, Q1 BC847C, Q2 BC847C, Q3 2N7002, SW1 SW_DPDT_x2, U1 SN74AHCT1G125DBVR, U10 ESP32-S3-WROOM-1-N4R2, U11 LDL1117S33R, U12 SN74CB3T3245PWR, U13 IS61C5128AS-25QLI, U2 SN74AHCT1G125DBVR, U3 LD1117S12, U4 SN74CB3T3245PWR, U5 MAX3221ECPWR, U6 XC6SLX9-2TQG144C, U7 Z84C3008VEG, U8 SN74CB3T3245PWR, U9 SN74CB3T3245PWR, X1 SX3M14.31818M20F30TNN

Commit message: Std rev3 PCB Updates
Parts:
- added C1: DNP, Capacitor_SMD:C_0603_1608Metric, F.Cu at (163.5, 59.8)
- added C2: DNP, Capacitor_SMD:C_0603_1608Metric, F.Cu at (167.5, 59.8)
- added JP3: vZ80 Enabled, Jumper:SolderJumper-2_P1.3mm_Bridged_RoundedPad1.0x1.5mm, F.Cu at (268.3, 75.5)
- added L1: USB Choke, Inductor_SMD:L_CommonMode_Wurth_WE-CNSW-1206, F.Cu at (165.5, 59.4)
- added R3: 0, Resistor_SMD:R_0603_1608Metric, F.Cu at (166.2, 63.2)
- added R4: 0, Resistor_SMD:R_0603_1608Metric, F.Cu at (164.8, 63.2)
- added U1: IP4234CZ6, Package_TO_SOT_SMD:SC-74-6_1.55x2.9mm_P0.95mm, F.Cu at (158.6, 58.6)
- FB1, FB2: value 220 -> 220o
- J11: renamed from J12; value Hand controller 1 -> Hand Controller
- J12: renamed from J11; value Hand controller 2 -> Hand Controller
- JP1, JP2: value USB -> Pin Header
- R38: renamed from R37; value 1 -> 0
- R40: renamed from R39; value 1 -> 0
- U3: renamed from U7; value Z84C3008VEG -> PLCC-44 SMD Socket
- moved C3 69.6 mm to (176.1, 61.0)
- moved R1 67.1 mm to (147.7, 64.2)
- moved R2 67.1 mm to (147.7, 65.7), turned to 0 degrees
- moved R28 66.8 mm to (253.5, 69.3)
- moved R23 66.8 mm to (249.0, 69.3)
- moved R24 66.8 mm to (247.5, 69.3)
- moved R25 66.8 mm to (250.5, 69.3)
- moved R26 66.8 mm to (255.0, 69.3)
- moved R27 66.8 mm to (252.0, 69.3)
- moved C19 65.5 mm to (190.2, 85.2)
- moved R62 65.5 mm to (263.0, 137.2)
- moved R64 65.5 mm to (264.4, 137.2)
- moved C11 65.5 mm to (153.8, 78.1)
- moved C16 65.5 mm to (180.3, 82.5)
- moved C32 65.5 mm to (179.8, 95.8)
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- renumbered C9 to C10, C8 to C12, C10 to C13, C25 to C14, C23 to C15, C12 to C16, C13 to C17, C14 to C18, C20 to C19, C17 to C20, C15 to C21, C16 to C22, C21 to C23, C19 to C24, C18 to C25, C22 to C26, C26 to C27, C27 to C29, C7 to C3, C29 to C30, C24 to C31, C36 to C33, C30 to C34, C34 to C35, C33 to C36, C31 to C38, C43 to C39, C1 to C4, C38 to C40, C39 to C41, C44 to C42, C40 to C43, C42 to C44, C41 to C45, C45 to C46, C49 to C47, C51 to C48, C35 to C49, C2 to C5, C52 to C51, C46 to C52, C47 to C55, C48 to C56, C55 to C57, C57 to C58, C58 to C59, C3 to C6, C56 to C60, C4 to C7, C5 to C8, C6 to C9, JP3 to JP5, R11 to R10, R7 to R11, R15 to R12, R16 to R13, R12 to R14, R8 to R15, R20 to R16, R13 to R17, R9 to R18, R21 to R19, R17 to R20, R10 to R21, R14 to R22, R24 to R23, R23 to R24, R28 to R26, R26 to R27, R27 to R28, R18 to R29, R32 to R30, R35 to R31, R33 to R32, R31 to R33, R29 to R34, R30 to R35, R34 to R36, R36 to R37, R38 to R39, R49 to R41, R68 to R42, R40 to R43, R41 to R44, R42 to R45, R43 to R46, R44 to R47, R45 to R48, R46 to R49, R3 to R5, R47 to R50, R48 to R51, R51 to R52, R50 to R53, R52 to R54, R54 to R55, R53 to R56, R55 to R57, R57 to R59, R5 to R6, R56 to R60, R59 to R61, R61 to R62, R60 to R63, R62 to R64, R64 to R65, R65 to R66, R63 to R67, R67 to R68, R66 to R69, R4 to R7, R69 to R70, R6 to R8, R19 to R9, U9 to U10, U12 to U11, U10 to U12, U11 to U13, U13 to U14, U3 to U4, U4 to U5, U1 to U6, U5 to U7, U6 to U8, U8 to U9
Connections:
- J10 pad 11: FPGA_EXP9 -> GND
- J2 pad 2: ESP_USB_D- -> Net-(J2-D-)
- J2 pad 3: ESP_USB_D+ -> Net-(J2-D+)
- JP1 pad 2: ESP_USB_D+ -> Net-(J2-D-)
- JP2 pad 2: ESP_USB_D- -> Net-(J2-D+)
- JP4 pad 1: Net-(JP4-Pin_1) -> GND
- JP4 pad 3: GND -> Net-(JP4-Pin_3)
- JP5 pad 1: Net-(JP3-A) -> GND
- JP5 pad 2: GND -> Net-(JP5-B)
- U12 pad 27: Net-(JP3-A) -> Net-(JP5-B)
- U12 pad 37: Net-(JP4-Pin_1) -> Net-(JP4-Pin_3)
- U8 pad 50: FPGA_EXP9 -> vZ80 Sense
Routing:
- net GND: track 133.6 -> 2006.1 mm, vias 248 -> 275
- net vZ80 Sense: track 0.00 -> 107.6 mm, vias 0 -> 4
- net FPGA_EXP9: track 50.2 -> 0.00 mm, vias 2 -> 0
- net Net-(J2-D-): track 0.00 -> 36.3 mm, vias 0 -> 1
- net Net-(J2-D+): track 0.00 -> 23.5 mm, vias 0 -> 1
- net ESP_USB_D+: track 87.5 -> 68.1 mm, vias 1 -> 2
- net ESP_USB_D-: track 85.3 -> 66.2 mm, vias 1 -> 2
- net Net-(J1-VBUS): track 8.63 -> 21.6 mm, vias 2 -> 3
- net /USB_D-: track 23.3 -> 11.6 mm
- net /USB_D+: track 23.3 -> 11.8 mm
- net Net-(JP3-A): track 10.3 -> 0.00 mm, vias 1 -> 0
- net Net-(JP5-B): track 0.00 -> 9.20 mm, vias 0 -> 1
- net Net-(L1-Pad3): track 0.00 -> 7.87 mm
- net Net-(JP4-Pin_3): track 0.00 -> 7.40 mm, vias 0 -> 1
- net Net-(JP4-Pin_1): track 7.20 -> 0.00 mm, vias 1 -> 0
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Other:
- board text added: "20240828"
- board text added: "Flash"
- board text added: "GND"
- board text added: "Rx"
- board text added: "Tx"
- board text added: "vZ"
- board text removed: "20240822"

Commit message: PCB folder updates and reorg
Parts:
- FB1, FB2: value 220o -> 220
Changed lines of the file:
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@@
 			(layer "F.SilkS"
 				(type "Top Silk Screen")
-				(color "White")
+				(color "#E1E1E1FF")
 			)
 			(layer "F.Paste"
@@
 			(layer "F.Mask"
 				(type "Top Solder Mask")
-				(color "#133C63D4")
+				(color "#213ED9E0")
 				(thickness 0.01)
 			)
@@
 			(layer "dielectric 1"
 				(type "core")
-				(thickness 1.51)
+				(color "FR4 natural")
+				(thickness 1.51 locked)
 				(material "FR4")
 				(epsilon_r 4.5)
@@
 			(layer "B.Mask"
 				(type "Bottom Solder Mask")
-				(color "#133C63D4")
+				(color "#213ED9E0")
 				(thickness 0.01)
 			)
@@
 			(layer "B.SilkS"
 				(type "Bottom Silk Screen")
-				(color "White")
+				(color "#E1E1E1FF")
 			)
 			(copper_finish "None")
@@
 		)
 		(property "Footprint" "aquarius-plus:CR22A-44D-2.54DSA(70)"
-			(at 0 0 -90)
+			(at 0 0 90)
 			(layer "F.Fab")
 			(hide yes)
@@
 		)
 		(property "Datasheet" ""
-			(at 0 0 -90)
+			(at 0 0 90)
 			(layer "F.Fab")
 			(hide yes)
@@
 		)
 		(property "Description" ""
-			(at 0 0 -90)
+			(at 0 0 90)
 			(layer "F.Fab")
 			(hide yes)
@@
 			(pintype "passive")
 		)
+		(model "${KIPRJMOD}/step/395-044-558-201-EDAC-Card-Edge-Connector.STEP"
+			(offset
+				(xyz -38.5 1.2 9.6)
+			)
+			(scale
+				(xyz 1 1 1)
+			)
+			(rotate
+				(xyz 0 0 0)
+			)
+		)
 	)
 	(footprint "Resistor_SMD:R_0603_1608Metric"
@@
 		(tags "resistor")
 		(property "Reference" "R50"
-			(at -1.50518 0.084111 270)
+			(at -1.50518 0.084111 -90)
 			(layer "F.SilkS")
 			(effects
@@
 		(tags "capacitor")
 		(property "Reference" "C52"
-			(at 1.672025 -0.109022 270)
+			(at 1.672025 -0.109022 -90)
 			(layer "F.SilkS")
 			(effects
@@
 		(tags "resistor")
 		(property "Reference" "R49"
-			(at -1.50448 0.07469 270)
+			(at -1.50448 0.07469 -90)
 			(layer "F.SilkS")
 			(effects
@@
 			)
 		)
-		(property "Value" "220o"
+		(property "Value" "220"
 			(at 0 1.43 0)
 			(layer "F.Fab")
@@
 			(thermal_bridge_angle 45)
 		)
+		(model "${KIPRJMOD}/step/PJ-3200.step"
+			(offset
+				(xyz 0 5 2.6)
+			)
+			(scale
+				(xyz 1 1 1)
+			)
+			(rotate
+				(xyz -90 0 180)
+			)
+		)
 	)
 	(footprint "Connector_PinHeader_2.54mm:PinHeader_2x06_P2.54mm_Vertical"
@@
 		(tags "resistor")
 		(property "Reference" "R47"
-			(at -1.48598 0.027203 270)
+			(at -1.48598 0.027203 -90)
 			(layer "F.SilkS")
 			(effects
@@
 			)
 		)
+		(model "${KIPRJMOD}/step/10118194-0001LF.stp"
+			(offset
+				(xyz -75 3.2 -0.4)
+			)
+			(scale
+				(xyz 1 1 1)
+			)
+			(rotate
+				(xyz 90 180 180)
+			)
+		)
 	)
 	(footprint "Resistor_SMD:R_0603_1608Metric"
@@
 			(thermal_bridge_angle 45)
 		)
+		(model "${KIPRJMOD}/step/PJ-3200.step"
+			(offset
+				(xyz 0 5 2.6)
+			)
+			(scale
+				(xyz 1 1 1)
+			)
+			(rotate
+				(xyz -90 0 180)
+			)
+		)
 	)
 	(footprint "Package_TO_SOT_SMD:SOT-23"
@@
 			(pintype "input")
 		)
+		(model "${KIPRJMOD}/step/SD Card Color.step"
+			(offset
+				(xyz 0 -13.5 0)
+			)
+			(scale
+				(xyz 1 1 1)
+			)
+			(rotate
+				(xyz -90 0 90)
+			)
+		)
 	)
 	(footprint "Package_TO_SOT_SMD:SOT-23-5"
@@
 		(tags "resistor")
 		(property "Reference" "R46"
-			(at -1.48958 0.040771 270)
+			(at -1.48958 0.040771 -90)
 			(layer "F.SilkS")
 			(effects
@@
 			(pintype "output")
 		)
-		(model "${KICAD8_3DMODEL_DIR}/Package_LCC.3dshapes/PLCC-44_SMD-Socket.wrl"
+		(model "${KIPRJMOD}/step/PLCC-44 SMD.step"
 			(offset
 				(xyz 0 0 0)
@@
 			)
 			(rotate
-				(xyz 0 0 0)
+				(xyz -90 0 90)
 			)
 		)
@@
 			(pintype "passive+no_connect")
 		)
-		(model "step/ICD15S13E4GV00LFc.stp"
+		(model "${KIPRJMOD}/step/ICD15S13E4GV00LFC.step"
 			(offset
 				(xyz 0 0.5 0)
@@
 			)
 			(rotate
-				(xyz 0 180 0)
+				(xyz 180 0 180)
 			)
 		)
@@
 		(tags "resistor")
 		(property "Reference" "R48"
-			(at -1.49958 -0.099428 270)
+			(at -1.49958 -0.099428 -90)
 			(layer "F.SilkS")
 			(effects
@@
 			(pintype "passive")
 		)
-		(model "${KICAD6_3DMODEL_DIR}/LED_THT.3dshapes/LED_D3.0mm_Horizontal_O1.27mm_Z2.0mm.wrl"
+		(model "${KIPRJMOD}/step/LED_D3.0mm_Horizontal_O1.27mm_Z2.0mm_Clear_Blue.step"
 			(offset
 				(xyz 0 0 0)
@@
 		)
 		(property "Value" "100"
-			(at 0 1.43 360)
+			(at 0 1.43 0)
 			(layer "F.Fab")
 			(effects
@@
 		)
 		(property "Footprint" "Resistor_SMD:R_0603_1608Metric"
-			(at 0 0 360)
+			(at 0 0 0)
 			(layer "F.Fab")
 			(hide yes)
@@
 		)
 		(property "Datasheet" ""
-			(at 0 0 360)
+			(at 0 0 0)
 			(layer "F.Fab")
 			(hide yes)
@@
 		)
 		(property "Description" ""
-			(at 0 0 360)
+			(at 0 0 0)
 			(layer "F.Fab")
 			(hide yes)
@@
 		)
 		(fp_text user "${REFERENCE}"
-			(at 0 0 360)
+			(at 0 0 0)
 			(layer "F.Fab")
 			(effects
@@
 			)
 		)
-		(property "Value" "220o"
+		(property "Value" "220"
 			(at 0 1.43 0)
 			(layer "F.Fab")
@@
 			(thermal_bridge_angle 45)
 		)
+		(model "${KIPRJMOD}/step/PJ-3200.step"
+			(offset
+				(xyz 0 5 2.6)
+			)
+			(scale
+				(xyz 1 1 1)
+			)
+			(rotate
+				(xyz 90 180 0)
+			)
+		)
 	)
 	(footprint "Resistor_SMD:R_0603_1608Metric"
@@
 		(tags "resistor")
 		(property "Reference" "R45"
-			(at -1.49868 0.027203 270)
+			(at -1.49868 0.027203 -90)
 			(layer "F.SilkS")
 			(effects
@@
 			(thermal_bridge_angle 45)
 		)
+		(model "${KIPRJMOD}/step/PJ-3200.step"
+			(offset
+				(xyz 0 5 2.6)
+			)
+			(scale
+				(xyz 1 1 1)
+			)
+			(rotate
+				(xyz -90 0 180)
+			)
+		)
 	)
 	(footprint "Capacitor_SMD:C_0805_2012Metric"
@@
 		(tags "resistor")
 		(property "Reference" "R44"
-			(at -1.50108 0.013636 270)
+			(at -1.50108 0.013636 -90)
 			(layer "F.SilkS")
 			(effects
@@
 		(min_thickness 0.2)
 		(filled_areas_thickness no)
-		(fill
+		(fill yes
 			(thermal_gap 0.3)
 			(thermal_bridge_width 0.3)

Commit message: Lots of updates...
Added Aq+ ICON images.
Reworked PCB directory.
Changed Mega project to Moda.
etc...
Parts:
- L1: footprint Inductor_SMD:L_CommonMode_Wurth_WE-CNSW-1206 -> Inductor_SMD_Wurth:WE-CNSW_08058
- moved L1 0.10 mm to (165.6, 59.4), turned to 0 degrees
Routing:
- net Net-(L1-Pad1): track 1.75 -> 2.33 mm
- net Net-(L1-Pad4): track 1.75 -> 2.25 mm
Other:
- board text added: "20240918"
- board text removed: "20240828"
Changed lines of the file:
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@@
 		)
 	)
-	(footprint "Inductor_SMD:L_CommonMode_Wurth_WE-CNSW-1206"
+	(footprint "Inductor_SMD_Wurth:WE-CNSW_08058"
 		(layer "F.Cu")
-		(at 165.5 59.35 90)
-		(descr "WE-CNSW SMT Common Mode Line Filter, https://www.we-online.com/components/products/datasheet/744232090.pdf")
-		(tags "common mode choke 1206 cnsw")
+		(at 165.6 59.35)
+		(descr "WE-CNSW_08058")
+		(tags "Inductor")
 		(property "Reference" "L1"
-			(at 3.029976 0.031121 0)
-			(unlocked yes)
+			(at 4.4 -0.85 0)
 			(layer "F.SilkS")
+			(hide yes)
 			(effects
 				(font
@@
 		)
 		(property "Value" "USB Choke"
-			(at 0 3.5 90)
-			(unlocked yes)
-			(layer "F.Fab")
+			(at -1.1712 1.5288 0)
+			(layer "F.SilkS")
+			(hide yes)
 			(effects
 				(font
-					(size 1 1)
-					(thickness 0.15)
+					(size 1.27 1.27)
+					(thickness 0.254)
 				)
 			)
 		)
-		(property "Footprint" "Inductor_SMD:L_CommonMode_Wurth_WE-CNSW-1206"
-			(at 0 0 90)
-			(unlocked yes)
+		(property "Footprint" "Inductor_SMD_Wurth:WE-CNSW_08058"
+			(at 0 0 0)
 			(layer "F.Fab")
 			(hide yes)
@@
 		)
 		(property "Datasheet" ""
-			(at 0 0 90)
-			(unlocked yes)
+			(at 0 0 0)
 			(layer "F.Fab")
 			(hide yes)
@@
 		)
 		(property "Description" "Common mode choke, 370 mA, 125VDC, USB2.0, 111 nH"
-			(at 0 0 90)
-			(unlocked yes)
+			(at 0 0 0)
 			(layer "F.Fab")
 			(hide yes)
@@
 		)
 		(property "JLCPCB" "C2649327"
-			(at 0 0 90)
+			(at 0 0 0)
 			(unlocked yes)
 			(layer "F.Fab")
@@
 		(attr smd)
 		(fp_line
-			(start -2.05 -1.05)
-			(end 1.35 -1.05)
+			(start -0.8 -1.5)
+			(end -0.8 1.5)
 			(stroke
-				(width 0.1)
-				(type default)
+				(width 0.127)
+				(type solid)
 			)
-			(layer "F.SilkS")
+			(layer "F.CrtYd")
 		)
 		(fp_line
-			(start -1.35 1.05)
-			(end 1.35 1.05)
+			(start -0.8 1.5)
+			(end 0.8 1.5)
 			(stroke
-				(width 0.1)
-				(type default)
+				(width 0.127)
+				(type solid)
 			)
-			(layer "F.SilkS")
+			(layer "F.CrtYd")
 		)
-		(fp_rect
-			(start -2.15 -1.05)
-			(end 2.15 1.05)
+		(fp_line
+			(start 0.8 -1.5)
+			(end -0.8 -1.5)
 			(stroke
-				(width 0.05)
-				(type default)
+				(width 0.127)
+				(type solid)
 			)
-			(fill none)
 			(layer "F.CrtYd")
 		)
 		(fp_line
-			(start 1.6 -0.8)
-			(end 1.6 0.8)
+			(start 0.8 1.5)
+			(end 0.8 -1.5)
 			(stroke
-				(width 0.1)
-				(type default)
+				(width 0.127)
+				(type solid)
+			)
+			(layer "F.CrtYd")
+		)
+		(fp_line
+			(start -0.6246 -1.2635)
+			(end 0.6251 -1.2635)
+			(stroke
+				(width 0.127)
+				(type solid)
 			)
 			(layer "F.Fab")
 		)
 		(fp_line
-			(start -1.1 -0.8)
-			(end 1.6 -0.8)
+			(start -0.6246 1.2874)
+			(end -0.6246 -1.2635)
 			(stroke
-				(width 0.1)
-				(type default)
+				(width 0.127)
+				(type solid)
 			)
 			(layer "F.Fab")
 		)
 		(fp_line
-			(start -1.6 -0.3)
-			(end -1.1 -0.8)
+			(start -0.4 -0.85)
+			(end -0.4 0.85)
 			(stroke
-				(width 0.1)
-				(type default)
+				(width 0.07)
+				(type solid)
 			)
 			(layer "F.Fab")
 		)
 		(fp_line
-			(start 1.6 0.8)
-			(end -1.6 0.8)
+			(start 0.4 -0.85)
+			(end 0.4 0.85)
 			(stroke
-				(width 0.1)
-				(type default)
+				(width 0.07)
+				(type solid)
 			)
 			(layer "F.Fab")
 		)
 		(fp_line
-			(start -1.6 0.8)
-			(end -1.6 -0.3)
+			(start 0.6203 1.2874)
+			(end -0.6246 1.2874)
 			(stroke
-				(width 0.1)
-				(type default)
+				(width 0.127)
+				(type solid)
+			)
+			(layer "F.Fab")
+		)
+		(fp_line
+			(start 0.6251 -1.2635)
+			(end 0.6251 1.2826)
+			(stroke
+				(width 0.127)
+				(type solid)
 			)
 			(layer "F.Fab")
 		)
 		(fp_text user "${REFERENCE}"
-			(at 0 0 90)
-			(unlocked yes)
+			(at 0.04316 -2.451663 0)
 			(layer "F.Fab")
 			(effects
 				(font
-					(size 0.7 0.7)
-					(thickness 0.105)
+					(size 1 1)
+					(thickness 0.15)
 				)
 			)
 		)
-		(pad "1" smd roundrect
-			(at -1.35 -0.5 90)
-			(size 1.1 0.6)
+		(pad "1" smd rect
+			(at -0.4 0.85)
+			(size 0.4 0.9)
 			(layers "F.Cu" "F.Paste" "F.Mask")
-			(roundrect_rratio 0.2)
 			(net 226 "Net-(L1-Pad1)")
 			(pintype "passive")
-			(thermal_bridge_angle 45)
 		)
-		(pad "2" smd roundrect
-			(at 1.35 -0.5 90)
-			(size 1.1 0.6)
+		(pad "2" smd rect
+			(at -0.4 -0.85)
+			(size 0.4 0.9)
 			(layers "F.Cu" "F.Paste" "F.Mask")
-			(roundrect_rratio 0.2)
 			(net 225 "Net-(L1-Pad2)")
 			(pintype "passive")
-			(thermal_bridge_angle 45)
 		)
-		(pad "3" smd roundrect
-			(at 1.35 0.5 90)
-			(size 1.1 0.6)
+		(pad "3" smd rect
+			(at 0.4 -0.85)
+			(size 0.4 0.9)
 			(layers "F.Cu" "F.Paste" "F.Mask")
-			(roundrect_rratio 0.2)
 			(net 224 "Net-(L1-Pad3)")
 			(pintype "passive")
-			(thermal_bridge_angle 45)
 		)
-		(pad "4" smd roundrect
-			(at -1.35 0.5 90)
-			(size 1.1 0.6)
+		(pad "4" smd rect
+			(at 0.4 0.85)
+			(size 0.4 0.9)
 			(layers "F.Cu" "F.Paste" "F.Mask")
-			(roundrect_rratio 0.2)
 			(net 227 "Net-(L1-Pad4)")
 			(pintype "passive")
-			(thermal_bridge_angle 45)
 		)
-		(model "${KICAD8_3DMODEL_DIR}/Inductor_SMD.3dshapes/L_CommonMode_Wurth_WE-CNSW-1206.wrl"
+		(model "744231091.stp"
 			(offset
-				(xyz 0 0 0)
+				(xyz 0 0 0.8099999902)
 			)
 			(scale
@@
 			)
 			(rotate
-				(xyz 0 0 0)
+				(xyz -180 0 90)
 			)
 		)
@@
 	)
 	(gr_circle
-		(center 164.072689 61.696853)
-		(end 164.372689 61.696853)
+		(center 164.586739 61.302029)
+		(end 164.886739 61.302029)
 		(stroke
 			(width 0.15)
@@
 		)
 	)
-	(gr_text "20240828"
+	(gr_text "20240918"
 		(at 132.578844 140.055462 90)
 		(layer "F.SilkS")
@@
 	)
 	(segment
-		(start 163.5 59)
-		(end 168.465045 59)
-		(width 0.3)
-		(layer "F.Cu")
-		(net 2)
-	)
-	(segment
 		(start 223.844436 84.7798)
 		(end 224.9341 84.7798)
@@
 	)
 	(segment
+		(start 168.084812 59.380233)
+		(end 168.465045 59)
+		(width 0.3)
+		(layer "F.Cu")
+		(net 2)
+	)
+	(segment
 		(start 144.798529 126.6998)
 		(end 144.05 126.6998)
@@
 	)
 	(segment
+		(start 163.880233 59.380233)
+		(end 168.084812 59.380233)
+		(width 0.3)
+		(layer "F.Cu")
+		(net 2)
+	)
+	(segment
 		(start 193.72 109.8248)
 		(end 193.72 108.587544)
@@
 	)
 	(segment
+		(start 163.5 59)
+		(end 163.880233 59.380233)
+		(width 0.3)
+		(layer "F.Cu")
+		(net 2)
+	)
+	(segment
 		(start 228.500772 77.666026)
 		(end 228.542997 77.623801)
@@
 	)
 	(segment
+		(start 166 57.45)
+		(end 166 58.5)
+		(width 0.2)
+		(layer "F.Cu")
+		(net 224)
+	)
+	(segment
 		(start 159.5 57.5)
 		(end 160.514044 56.485956)
@@
 	)
 	(segment
-		(start 166 57.45)
-		(end 166 58)
-		(width 0.2)
-		(layer "F.Cu")
-		(net 224)
-	)
-	(segment
 		(start 160.514044 56.485956)
 		(end 165.035956 56.485956)
@@
 	)
 	(segment
-		(start 162.129748 58)
-		(end 160.329748 59.8)
+		(start 161.1 58.2)
+		(end 159.5 59.8)
 		(width 0.3)
 		(layer "F.Cu")
@@
 	)
 	(segment
-		(start 165 58)
-		(end 162.129748 58)
+		(start 165.2 58.5)
+		(end 164.9 58.2)
 		(width 0.3)
 		(layer "F.Cu")
@@
 	)
 	(segment
-		(start 160.329748 59.8)
-		(end 159.5 59.8)
+		(start 164.9 58.2)
+		(end 161.1 58.2)
 		(width 0.3)
 		(layer "F.Cu")
@@
 	)
 	(segment
-		(start 165 62.110119)
-		(end 164.76181 62.348309)
+		(start 165.2 60.2)
+		(end 165.2 61.910119)
 		(width 0.3)
 		(layer "F.Cu")
@@
 	)
 	(segment
-		(start 165 60.7)
-		(end 165 62.110119)
+		(start 165.2 61.910119)
+		(end 164.76181 62.348309)
 		(width 0.3)
 		(layer "F.Cu")
@@
 	)
 	(segment
-		(start 166 60.7)
+		(start 166 60.2)
 		(end 166 62.10206)
 		(width 0.3)
@@
 		(min_thickness 0.2)
 		(filled_areas_thickness no)
-		(fill yes
+		(fill
 			(thermal_gap 0.3)
 			(thermal_bridge_width 0.3)

Commit message: Standard PCB rev3 updates in anticipation of prototype build
Parts:
- added J22: Conn_01x04_Pin, Connector_PinHeader_2.54mm:PinHeader_1x04_P2.54mm_Vertical, F.Cu at (172.5, 46.8)
Routing:
- net GND: track 2006.4 -> 2016.1 mm
- net Net-(J2-D+): track 23.5 -> 28.7 mm
- net Net-(J2-VBUS): track 9.42 -> 14.6 mm
- net Net-(J2-D-): track 36.3 -> 41.4 mm
Other:
- board text added: "Requires a Z80 CMOS CPU PLCC44 10MHZ or higher Z84C0010VEC"
- board text removed: "vZ"
