File: standard/rev3/aquarius-plus.kicad_sch (KiCad schematic)
At the start: 173 parts, among them J1 Power in, J10 FPGA spare, J11 Hand controller 2, J12 Hand controller 1, J13 ESP32 spare, J2 ESP USB Host, J3 Audio out, J4 VGA, J5 Cassette out, J6 Cassette in, J7 Expansion port, J8 Printer, J9 TF-03A, Q1 BC847C, Q2 BC847C, Q3 2N7002, SW1 SW_DPDT_x2, U1 SN74AHCT1G125DBVR, U10 ESP32-S3-WROOM-1-N4R2, U11 LDL1117S33R, U12 SN74CB3T3245PWR, U13 IS61C5128AS-25QLI, U2 SN74AHCT1G125DBVR, U3 LD1117S12, U4 SN74CB3T3245PWR, U5 MAX3221ECPWR, U6 XC6SLX9-2TQG144C, U7 Z84C3008VEG, U8 SN74CB3T3245PWR, U9 SN74CB3T3245PWR, X1 SX3M14.31818M20F30TNN

Commit message: Std rev3 PCB Updates
Parts:
- added C1, C2: DNP, Capacitor_SMD:C_0603_1608Metric, symbol Device:C_Small
- added JP3: vZ80 Enabled, Jumper:SolderJumper-2_P1.3mm_Bridged_RoundedPad1.0x1.5mm, symbol Jumper:SolderJumper_2_Bridged
- added L1: USB Choke, Inductor_SMD:L_CommonMode_Wurth_WE-CNSW-1206, symbol Filter:Choke_Wurth_WE-CNSW_744232090
- added R3, R4: 0, Resistor_SMD:R_0603_1608Metric, symbol Device:R
- added U1: IP4234CZ6, Package_TO_SOT_SMD:SC-74-6_1.55x2.9mm_P0.95mm, symbol Power_Protection:IP4234CZ6
- C10: renamed from C9; JLCPCB (none) -> C14663
- C11, C50, C53: JLCPCB (none) -> C19666
- C12: renamed from C8; JLCPCB (none) -> C14663
- C13: renamed from C10; JLCPCB (none) -> C14663
- C14: renamed from C25; JLCPCB (none) -> C14663
- C15: renamed from C23; JLCPCB (none) -> C19666
- C16: renamed from C12; JLCPCB (none) -> C19666
- C17: renamed from C13; JLCPCB (none) -> C19666
- C18: renamed from C14; JLCPCB (none) -> C14663
- C19: renamed from C20; JLCPCB (none) -> C19666
- C20: renamed from C17; JLCPCB (none) -> C14663
- C21: renamed from C15; JLCPCB (none) -> C14663
- C22: renamed from C16; JLCPCB (none) -> C14663
- C23: renamed from C21; JLCPCB (none) -> C19666
- C24: renamed from C19; JLCPCB (none) -> C14663
- C25: renamed from C18; JLCPCB (none) -> C14663
- C26: renamed from C22; JLCPCB (none) -> C14663
- C27: renamed from C26; JLCPCB (none) -> C14663
- C28, C32, C37, C54: JLCPCB (none) -> C14663
- C29: renamed from C27; JLCPCB (none) -> C14663
- C3: renamed from C7; JLCPCB (none) -> C264047
- C30: renamed from C29; JLCPCB (none) -> C14663
- C31: renamed from C24; JLCPCB (none) -> C14663
- C33: renamed from C36; JLCPCB (none) -> C14663
- C34: renamed from C30; JLCPCB (none) -> C14663
- C35: renamed from C34; JLCPCB (none) -> C19666
- C36: renamed from C33; JLCPCB (none) -> C19666
- C38: renamed from C31; JLCPCB (none) -> C14663
- C39: renamed from C43; JLCPCB (none) -> C14663
- C4: renamed from C1; JLCPCB (none) -> C15850
- C40: renamed from C38; JLCPCB (none) -> C14663
- C41: renamed from C39; JLCPCB (none) -> C14663
- C42: renamed from C44; JLCPCB (none) -> C19666
- C43: renamed from C40; JLCPCB (none) -> C14663
- C44: renamed from C42; JLCPCB (none) -> C14663
- C45: renamed from C41; JLCPCB (none) -> C14663
- C46: renamed from C45; JLCPCB (none) -> C14663
- C47: renamed from C49; JLCPCB (none) -> C14663
- C48: renamed from C51; JLCPCB (none) -> C14663
- C49: renamed from C35; JLCPCB (none) -> C19666
- C5: renamed from C2; JLCPCB (none) -> C14663
- C51: renamed from C52; JLCPCB (none) -> C14663
- C52: renamed from C46; JLCPCB (none) -> C14663
- C55: renamed from C47; JLCPCB (none) -> C19666
- C56: renamed from C48; JLCPCB (none) -> C19666
- C57: renamed from C55; JLCPCB (none) -> C14663
- C58: renamed from C57; JLCPCB (none) -> C14663
- C59: renamed from C58; JLCPCB (none) -> C12891
- C6: renamed from C3; JLCPCB (none) -> C15850
- C60: renamed from C56; JLCPCB (none) -> C19666
- C7: renamed from C4; JLCPCB (none) -> C14663
- C8: renamed from C5; JLCPCB (none) -> C264047
- C9: renamed from C6; JLCPCB (none) -> C14663
- D1, D2: JLCPCB (none) -> C2128
- D3: JLCPCB (none) -> C330760
- FB1, FB2: JLCPCB (none) -> C2661695
- FID1, FID2, FID3: now not fitted
- H1, H2, H3, H4, J10, J13, JP4: now not fitted; now left out of the parts list
- J1: JLCPCB (none) -> C132563
- J11: renamed from J12; value Hand controller 1 -> Hand Controller; JLCPCB (none) -> C305940
- J12: renamed from J11; value Hand controller 2 -> Hand Controller; JLCPCB (none) -> C305940
- J2: JLCPCB (none) -> C2798029
- J3, J5, J6, J8: JLCPCB (none) -> C2939180
- J4: JLCPCB (none) -> C138387
- J7: JLCPCB (none) -> C7431259
- J9: JLCPCB (none) -> C693842
- JP1, JP2: value USB -> Pin Header; JLCPCB (none) -> C5116481
- JP5: renamed from JP3; JLCPCB (none) -> C5116481
- Q1, Q2: JLCPCB (none) -> C181141
- Q3: JLCPCB (none) -> C8545
- R1: JLCPCB (none) -> C25804
- R10: renamed from R11; JLCPCB (none) -> C137783
- R11: renamed from R7; JLCPCB (none) -> C227956
- R12: renamed from R15; JLCPCB (none) -> C170518
- R13: renamed from R16; JLCPCB (none) -> C170518
- R14: renamed from R12; JLCPCB (none) -> C137783
- R15: renamed from R8; JLCPCB (none) -> C227956
- R16: renamed from R20; JLCPCB (none) -> C23159
- R17: renamed from R13; JLCPCB (none) -> C137783
- R18: renamed from R9; JLCPCB (none) -> C227956
- R19: renamed from R21; JLCPCB (none) -> C23159
- R2, R58: JLCPCB (none) -> C22775
- R20: renamed from R17; JLCPCB (none) -> C170518
- R21: renamed from R10; JLCPCB (none) -> C23253
- R22: renamed from R14; JLCPCB (none) -> C23253
- R23: renamed from R24; JLCPCB (none) -> C21190
- R24: renamed from R23; JLCPCB (none) -> C21190
- R25: JLCPCB (none) -> C21190
- R26: renamed from R28; JLCPCB (none) -> C21190
- R27: renamed from R26; JLCPCB (none) -> C21190
- R28: renamed from R27; JLCPCB (none) -> C21190
- R29: renamed from R18; JLCPCB (none) -> C23255
- R30: renamed from R32; JLCPCB (none) -> C25819
- R31: renamed from R35; JLCPCB (none) -> C25819
- R32: renamed from R33; JLCPCB (none) -> C22962
- R33: renamed from R31; JLCPCB (none) -> C22961
- R34: renamed from R29; JLCPCB (none) -> C23162
- R35: renamed from R30; JLCPCB (none) -> C23162
- R36: renamed from R34; JLCPCB (none) -> C4190
- R37: renamed from R36; JLCPCB (none) -> C22775
- R38: renamed from R37; value 1 -> 0; JLCPCB (none) -> C2784885
- R39: renamed from R38; JLCPCB (none) -> C22962
- R40: renamed from R39; value 1 -> 0; JLCPCB (none) -> C2784885
- R41: renamed from R49; JLCPCB (none) -> C25804
- R42: renamed from R68; JLCPCB (none) -> C25804
- R43: renamed from R40; JLCPCB (none) -> C25804
- R44: renamed from R41; JLCPCB (none) -> C22775
- R45: renamed from R42; JLCPCB (none) -> C25804
- R46: renamed from R43; JLCPCB (none) -> C22775
- R47: renamed from R44; JLCPCB (none) -> C25804
- R48: renamed from R45; JLCPCB (none) -> C22775
- R49: renamed from R46; JLCPCB (none) -> C22775
- R5: renamed from R3; JLCPCB (none) -> C22808
- R50: renamed from R47; JLCPCB (none) -> C25804
- R51: renamed from R48; JLCPCB (none) -> C25804
- R52: renamed from R51; JLCPCB (none) -> C22775
- R53: renamed from R50; JLCPCB (none) -> C22775
- R54: renamed from R52; JLCPCB (none) -> C22775
- R55: renamed from R54; JLCPCB (none) -> C22775
- R56: renamed from R53; JLCPCB (none) -> C22775
- R57: renamed from R55; JLCPCB (none) -> C22775
- R59: renamed from R57; JLCPCB (none) -> C22775
- R6: renamed from R5; JLCPCB (none) -> C22808
- R60: renamed from R56; JLCPCB (none) -> C22775
- R61: renamed from R59; JLCPCB (none) -> C22775
- R62: renamed from R61; JLCPCB (none) -> C22775
- R63: renamed from R60; JLCPCB (none) -> C22775
- R64: renamed from R62; JLCPCB (none) -> C22775
- R65: renamed from R64; JLCPCB (none) -> C22775
- R66: renamed from R65; JLCPCB (none) -> C22775
- R67: renamed from R63; JLCPCB (none) -> C22775
- R68: renamed from R67; JLCPCB (none) -> C22775
- R69: renamed from R66; JLCPCB (none) -> C22775
- R7: renamed from R4; JLCPCB (none) -> C23138
- R70: renamed from R69; JLCPCB (none) -> C22962
- R8: renamed from R6; JLCPCB (none) -> C23138
- R9: renamed from R19; JLCPCB (none) -> C23159
- SW1: JLCPCB (none) -> C3664594
- U10: renamed from U9; JLCPCB (none) -> C15298
- U11: renamed from U12; JLCPCB (none) -> C15298
- U12: renamed from U10; JLCPCB (none) -> C2913203
- U13: renamed from U11; JLCPCB (none) -> C155612
- U14: renamed from U13; JLCPCB (none) -> C443416
- U2: JLCPCB (none) -> C7484
- U3: renamed from U7; value Z84C3008VEG -> PLCC-44 SMD Socket; JLCPCB (none) -> C2828044
- U4: renamed from U3; JLCPCB (none) -> C155612
- U5: renamed from U4; JLCPCB (none) -> C15298
- U6: renamed from U1; JLCPCB (none) -> C7484
- U7: renamed from U5; JLCPCB (none) -> C350553
- U8: renamed from U6; JLCPCB (none) -> C27408
- U9: renamed from U8; JLCPCB (none) -> C15298
- X1: JLCPCB (none) -> C2901565
Connections:
- net ESP_USB_D+: now also C1.2, R4.2; no longer J2.3 (D+), JP1.2 (B)
- net ESP_USB_D-: now also C2.2, R3.2; no longer J2.2 (D-), JP2.2 (B)
- net GND: now also J10.11 (Pin_11), JP4.1 (Pin_1), JP5.1 (A), C1.1, C2.1, JP3.1 (A), U1.2 (VN); no longer JP4.3 (Pin_3), JP5.2 (B)
- net at FB1.1, J1.1 (VBUS): now also U1.5 (VP)
- net at U12.27 (IO0): now also JP5.2 (B); no longer JP5.1 (A)
- net at U12.37 (IO43/TXD0): now also JP4.3 (Pin_3); no longer JP4.1 (Pin_1)
- net FPGA_EXP9 renamed vZ80 Sense
- net vZ80 Sense: now also JP3.2 (B); no longer J10.11 (Pin_11)
- new net: J2.3 (D+), JP2.2 (B), U1.6
- new net: J2.2 (D-), JP1.2 (B), U1.1
- new net: L1.2, U1.3
- new net: L1.3, U1.4
- new net: L1.4, R3.1
- new net: L1.1, R4.1
Other:
- moved on the sheet: C16, C17, C3, C4, C5, C55, C56, C6, C7, C8, FB1, FB2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

Commit message: Lots of updates...
Added Aq+ ICON images.
Reworked PCB directory.
Changed Mega project to Moda.
etc...
Parts:
- L1: footprint Inductor_SMD:L_CommonMode_Wurth_WE-CNSW-1206 -> Inductor_SMD_Wurth:WE-CNSW_08058
Changed lines of the file:
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@@
 			)
 		)
-		(property "Footprint" "Inductor_SMD:L_CommonMode_Wurth_WE-CNSW-1206"
+		(property "Footprint" "Inductor_SMD_Wurth:WE-CNSW_08058"
 			(at 490.22 143.51 0)
 			(effects

Commit message: Standard PCB rev3 updates in anticipation of prototype build
Parts:
- added J22: Conn_01x04_Pin, Connector_PinHeader_2.54mm:PinHeader_1x04_P2.54mm_Vertical, symbol Connector:Conn_01x04_Pin
Connections:
- net GND: now also J22.4 (Pin_4)
- net at J2.3 (D+), JP2.2 (B), U1.6: now also J22.3 (Pin_3)
- net at J2.2 (D-), JP1.2 (B), U1.1: now also J22.2 (Pin_2)
- net at FB2.1, J2.1 (VBUS): now also J22.1 (Pin_1)
Changed lines of the file:
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@@
 	)
 	(junction
+		(at 444.5 121.92)
+		(diameter 0)
+		(color 0 0 0 0)
+	)
+	(junction
 		(at 130.81 91.44)
 		(diameter 0)
@@
 	)
 	(junction
+		(at 434.34 138.43)
+		(diameter 0)
+		(color 0 0 0 0)
+	)
+	(junction
 		(at 153.67 259.08)
 		(diameter 0)
@@
 	)
 	(junction
+		(at 445.77 129.54)
+		(diameter 0)
+		(color 0 0 0 0)
+	)
+	(junction
 		(at 128.27 313.69)
 		(diameter 0)
@@
 	)
 	(junction
+		(at 443.23 127)
+		(diameter 0)
+		(color 0 0 0 0)
+	)
+	(junction
 		(at 21.59 314.96)
 		(diameter 0)
@@
 	(wire
 		(pts
+			(xy 453.39 142.24) (xy 445.77 142.24)
+		)
+		(stroke
+			(width 0)
+			(type default)
+		)
+	)
+	(wire
+		(pts
 			(xy 261.62 203.2) (xy 264.16 203.2)
 		)
@@
 	(wire
 		(pts
+			(xy 453.39 147.32) (xy 438.15 147.32)
+		)
+		(stroke
+			(width 0)
+			(type default)
+		)
+	)
+	(wire
+		(pts
 			(xy 44.45 335.28) (xy 55.88 335.28)
 		)
@@
 	(wire
 		(pts
+			(xy 445.77 129.54) (xy 471.17 129.54)
+		)
+		(stroke
+			(width 0)
+			(type default)
+		)
+	)
+	(wire
+		(pts
 			(xy 187.96 120.65) (xy 187.96 121.92)
 		)
@@
 	(wire
 		(pts
-			(xy 441.96 129.54) (xy 471.17 129.54)
+			(xy 441.96 129.54) (xy 445.77 129.54)
 		)
 		(stroke
@@
 	(wire
 		(pts
+			(xy 443.23 144.78) (xy 453.39 144.78)
+		)
+		(stroke
+			(width 0)
+			(type default)
+		)
+	)
+	(wire
+		(pts
 			(xy 191.77 99.06) (xy 191.77 100.33)
 		)
@@
 	(wire
 		(pts
+			(xy 434.34 138.43) (xy 438.15 138.43)
+		)
+		(stroke
+			(width 0)
+			(type default)
+		)
+	)
+	(wire
+		(pts
 			(xy 236.22 287.02) (xy 231.14 287.02)
 		)
@@
 	(wire
 		(pts
-			(xy 441.96 127) (xy 468.63 127)
+			(xy 444.5 121.92) (xy 445.77 121.92)
+		)
+		(stroke
+			(width 0)
+			(type default)
+		)
+	)
+	(wire
+		(pts
+			(xy 441.96 127) (xy 443.23 127)
 		)
 		(stroke
@@
 	(wire
 		(pts
+			(xy 444.5 121.92) (xy 444.5 139.7)
+		)
+		(stroke
+			(width 0)
+			(type default)
+		)
+	)
+	(wire
+		(pts
 			(xy 304.8 144.78) (xy 313.69 144.78)
 		)
@@
 	(wire
 		(pts
-			(xy 441.96 121.92) (xy 445.77 121.92)
+			(xy 441.96 121.92) (xy 444.5 121.92)
 		)
 		(stroke
@@
 	(wire
 		(pts
+			(xy 443.23 127) (xy 443.23 144.78)
+		)
+		(stroke
+			(width 0)
+			(type default)
+		)
+	)
+	(wire
+		(pts
 			(xy 477.52 123.19) (xy 477.52 135.89)
 		)
@@
 		)
 	)
+	(wire
+		(pts
+			(xy 438.15 147.32) (xy 438.15 138.43)
+		)
+		(stroke
+			(width 0)
+			(type default)
+		)
+	)
 	(polyline
 		(pts
@@
 	(wire
 		(pts
+			(xy 443.23 127) (xy 468.63 127)
+		)
+		(stroke
+			(width 0)
+			(type default)
+		)
+	)
+	(wire
+		(pts
 			(xy 210.82 252.73) (xy 209.55 252.73)
 		)
@@
 		)
 	)
+	(wire
+		(pts
+			(xy 444.5 139.7) (xy 453.39 139.7)
+		)
+		(stroke
+			(width 0)
+			(type default)
+		)
+	)
 	(polyline
 		(pts
@@
 	(wire
 		(pts
+			(xy 445.77 142.24) (xy 445.77 129.54)
+		)
+		(stroke
+			(width 0)
+			(type default)
+		)
+	)
+	(wire
+		(pts
 			(xy 196.85 113.03) (xy 196.85 100.33)
 		)
@@
 					(unit 1)
 				)
+			)
+		)
+	)
+	(symbol
+		(lib_id "Connector:Conn_01x04_Pin")
+		(at 458.47 142.24 0)
+		(mirror y)
+		(unit 1)
+		(exclude_from_sim no)
+		(in_bom yes)
+		(on_board yes)
+		(dnp no)
+		(property "Reference" "J22"
+			(at 457.835 134.62 0)
+			(effects
+				(font
+					(size 1.27 1.27)
+				)
+			)
+		)
+		(property "Value" "Conn_01x04_Pin"
+			(at 457.835 137.16 0)
+			(effects
+				(font
+					(size 1.27 1.27)
+				)
+			)
+		)
+		(property "Footprint" "Connector_PinHeader_2.54mm:PinHeader_1x04_P2.54mm_Vertical"
+			(at 458.47 142.24 0)
+			(effects
+				(font
+					(size 1.27 1.27)
+				)
+				(hide yes)
+			)
+		)
+		(property "Datasheet" "~"
+			(at 458.47 142.24 0)
+			(effects
+				(font
+					(size 1.27 1.27)
+				)
+				(hide yes)
+			)
+		)
+		(property "Description" "Generic connector, single row, 01x04, script generated"
+			(at 458.47 142.24 0)
+			(effects
+				(font
+					(size 1.27 1.27)
+				)
+				(hide yes)
+			)
+		)
+		(pin "4"
+		)
+		(pin "3"
+		)
+		(pin "2"
+		)
+		(pin "1"
+		)
+		(instances
+			(project ""
+				(path "/e63e39d7-6ac0-4ffd-8aa3-1841a4541b55"
+					(reference "J22")
+					(unit 1)
+				)
